File: Hardware/Elektrische_Komm.sch (KiCad schematic (older format))
At the start: 93 parts

Commit message: same
Parts:
- added C?: 100n, Capacitors_SMD:C_0603, symbol C
- added C?: 470n, Capacitors_SMD:C_0603, symbol C
- added D?: LED_ALT, symbol LED_ALT
- added R?: R, Resistors_SMD:R_0603, symbol R
- added U?: LDK715M50R, TO_SOT_Packages_SMD:SOT-23-5_HandSoldering, symbol LDK715M50R
- U?: footprint (none) -> TO_SOT_Packages_SMD:SOT-23-6
Connections:
- net +15V: now also C?.1, U?.4 (VIN)
- net +3V3: now also R?.1
- net +5V: now also C?.1, U?.5 (VOUT)
- net GNDREF: now also C?.2, C?.2, D?.1 (K), U?.2 (GND)
- new net: D?.2 (A), R?.2
Other:
- note added: "Spannungsregler"
Changed lines of the file:
@@
 	4400 2500 4400 5950
 Wire Notes Line
-	450  5950 10800 5950
+	450  5950 19200 5950
 Wire Wire Line
 	5700 1250 6100 1250
@@
 F 0 "U?" H 12900 6950 60  0000 C CNN
 F 1 "TPS561201" H 12900 6850 60  0000 C CNN
-F 2 "" H 12900 7000 60  0001 C CNN
+F 2 "TO_SOT_Packages_SMD:SOT-23-6" H 12900 7000 60  0001 C CNN
 F 3 "" H 12900 7000 60  0001 C CNN
 	1    12900 7000
@@
 	0    1    1    0
 $EndComp
+Wire Notes Line
+	19200 5950 19200 7850
+Wire Notes Line
+	19200 7850 10800 7850
+Text Notes 11000 7750 0    157  ~ 0
+Spannungsregler
+$Comp
+L R R?
+U 1 1 5AFA2D21
+P 10300 11700
+F 0 "R?" V 10380 11700 50  0000 C CNN
+F 1 "R" V 10300 11700 50  0000 C CNN
+F 2 "Resistors_SMD:R_0603" V 10230 11700 50  0001 C CNN
+F 3 "" H 10300 11700 50  0001 C CNN
+	1    10300 11700
+	1    0    0    -1
+$EndComp
+$Comp
+L +3.3V #PWR?
+U 1 1 5AFA2EBF
+P 10300 11400
+F 0 "#PWR?" H 10300 11250 50  0001 C CNN
+F 1 "+3.3V" H 10300 11540 50  0000 C CNN
+F 2 "" H 10300 11400 50  0001 C CNN
+F 3 "" H 10300 11400 50  0001 C CNN
+	1    10300 11400
+	1    0    0    -1
+$EndComp
+Wire Wire Line
+	10300 11400 10300 11550
+$Comp
+L LED_ALT D?
+U 1 1 5AFA31A8
+P 10300 12000
+F 0 "D?" H 10300 12100 50  0000 C CNN
+F 1 "LED_ALT" H 10300 11900 50  0000 C CNN
+F 2 "" H 10300 12000 50  0001 C CNN
+F 3 "" H 10300 12000 50  0001 C CNN
+	1    10300 12000
+	0    -1   -1   0
+$EndComp
+$Comp
+L GNDREF #PWR?
+U 1 1 5AFA328E
+P 10300 12300
+F 0 "#PWR?" H 10300 12050 50  0001 C CNN
+F 1 "GNDREF" H 10300 12150 50  0000 C CNN
+F 2 "" H 10300 12300 50  0001 C CNN
+F 3 "" H 10300 12300 50  0001 C CNN
+	1    10300 12300
+	1    0    0    -1
+$EndComp
+Wire Wire Line
+	10300 12300 10300 12150
+$Comp
+L LDK715M50R U?
+U 1 1 5AFA4CE5
+P 17050 6950
+F 0 "U?" H 17150 7050 61  0000 C CNN
+F 1 "LDK715M50R" H 17350 6950 61  0000 C CNN
+F 2 "TO_SOT_Packages_SMD:SOT-23-5_HandSoldering" H 17050 6950 157 0001 C CNN
+F 3 "" H 17050 6950 157 0001 C CNN
+	1    17050 6950
+	1    0    0    -1
+$EndComp
+$Comp
+L GNDREF #PWR?
+U 1 1 5AFA54CF
+P 16900 7300
+F 0 "#PWR?" H 16900 7050 50  0001 C CNN
+F 1 "GNDREF" H 16900 7150 50  0000 C CNN
+F 2 "" H 16900 7300 50  0001 C CNN
+F 3 "" H 16900 7300 50  0001 C CNN
+	1    16900 7300
+	1    0    0    -1
+$EndComp
+$Comp
+L C C?
+U 1 1 5AFA5603
+P 16400 6950
+F 0 "C?" H 16425 7050 50  0000 L CNN
+F 1 "100n" H 16425 6850 50  0000 L CNN
+F 2 "Capacitors_SMD:C_0603" H 16438 6800 50  0001 C CNN
+F 3 "" H 16400 6950 50  0001 C CNN
+	1    16400 6950
+	1    0    0    -1
+$EndComp
+$Comp
+L C C?
+U 1 1 5AFA5A66
+P 17800 6950
+F 0 "C?" H 17825 7050 50  0000 L CNN
+F 1 "470n" H 17825 6850 50  0000 L CNN
+F 2 "Capacitors_SMD:C_0603" H 17838 6800 50  0001 C CNN
+F 3 "" H 17800 6950 50  0001 C CNN
+	1    17800 6950
+	1    0    0    -1
+$EndComp
+$Comp
+L +15V #PWR?
+U 1 1 5AFA5B62
+P 16050 6500
+F 0 "#PWR?" H 16050 6350 50  0001 C CNN
+F 1 "+15V" H 16050 6640 50  0000 C CNN
+F 2 "" H 16050 6500 50  0001 C CNN
+F 3 "" H 16050 6500 50  0001 C CNN
+	1    16050 6500
+	0    -1   -1   0
+$EndComp
+Wire Wire Line
+	16050 6500 16450 6500
+Wire Wire Line
+	16400 6800 16400 6500
+Connection ~ 16400 6500
+$Comp
+L +5V #PWR?
+U 1 1 5AFA5FD0
+P 18000 6500
+F 0 "#PWR?" H 18000 6350 50  0001 C CNN
+F 1 "+5V" H 18000 6640 50  0000 C CNN
+F 2 "" H 18000 6500 50  0001 C CNN
+F 3 "" H 18000 6500 50  0001 C CNN
+	1    18000 6500
+	0    1    1    0
+$EndComp
+Wire Wire Line
+	18000 6500 17350 6500
+Wire Wire Line
+	17800 6800 17800 6500
+Connection ~ 17800 6500
+Wire Wire Line
+	16900 6900 16900 7300
+Wire Wire Line
+	16400 7100 16400 7200
+Wire Wire Line
+	16400 7200 17800 7200
+Connection ~ 16900 7200
+Wire Wire Line
+	17800 7200 17800 7100
+Wire Notes Line
+	11400 5950 11400 450
 $EndSCHEMATC

Commit message: ACS723-Datenblatt
Parts:
- added C? (x5): 1µ, Capacitors_SMD:C_0603, symbol C
- added C?: 4,7µ, Capacitors_SMD:C_0603, symbol C
- added C? (x2): 20p, Capacitors_SMD:C_0603, symbol C
- added J? (x3): Conn_01x01, symbol Conn_01x01
- added R?: 1k, Resistors_SMD:R_0603, symbol R
- added SW?: SW_Push, symbol SW_Push
- added TP? (x15): TEST, Pin_Headers:Pin_Header_Straight_1x01_Pitch1.00mm, symbol TEST
- added U? (x8): STM32F413R(G-H)Tx_u, LQFP64, symbol STM32F413R(G-H)Tx_u
- added Y?: 10MHz, symbol Crystal_Small
Connections:
- net +15V: now also Q?.3 (D), Q?.3 (D), Q?.3 (D), TP?.1
- net +3V3: now also R?.1, TP?.1
- net +5V: now also TP?.1
- net A_conn: now also J?.1 (Pin_1), TP?.1
- net B_conn: now also J?.1 (Pin_1), TP?.1
- net Bemf_A: now also U?.41 (PA8/CAN3_RX/DFSDM1_CKOUT/I2C3_SCL/RCC_MCO_1/SDIO_D1/TIM1_CH1/UART7_RX/USART1_CK/USB_OTG_FS_SOF)
- net Bemf_B: now also U?.42 (PA9/DAC_EXTI9/DFSDM2_CKIN3/I2C3_SMBA/I2S2_CK/SDIO_D2/SPI2_SCK/TIM1_CH2/USART1_TX/USB_OTG_FS_VBUS)
- net Bemf_C: now also U?.43 (PA10/DFSDM2_DATIN3/I2S2_SD/I2S5_SD/SPI2_MOSI/SPI5_MOSI/TIM1_CH3/USART1_RX/USB_OTG_FS_ID)
- net C: now also J?.1 (Pin_1), TP?.1
- net Curr_direct_A: now also TP?.1
- net Curr_direct_B: now also TP?.1
- net Curr_mcu_A: now also U?.8 (PC0/ADC1_IN10/DFSDM2_CKIN4/LPTIM1_IN1/SAI1_MCLK_B/SYS_WKUP2)
- net Curr_mcu_B: now also U?.9 (PC1/ADC1_IN11/DFSDM2_DATIN4/LPTIM1_OUT/SAI1_SD_B/SYS_WKUP3)
- net GNDREF: now also C?.1, C?.1, C?.1, C?.1, C?.1, C?.1, C?.1, C?.1, SW?.2, TP?.1, TP?.1, TP?.1, U?.12 (VSSA), U?.18 (VSS), U?.31 (VSS), U?.47 (VSS), U?.60 (BOOT0), U?.63 (VSS)
- net HI_A: now also U?.22 (PA6/ADC1_IN6/DFSDM2_CKIN1/I2S2_MCK/QUADSPI_BK2_IO0/SDIO_CMD/SPI1_MISO/TIM13_CH1/TIM1_BKIN/TIM3_CH1/TIM8_BKIN)
- net HI_B: now also U?.23 (PA7/ADC1_IN7/DFSDM2_DATIN1/I2S1_SD/QUADSPI_BK2_IO1/SPI1_MOSI/TIM14_CH1/TIM1_CH1N/TIM3_CH2/TIM8_CH1N)
- net HI_C: now also U?.26 (PB0/ADC1_IN8/I2S5_CK/SPI5_SCK/TIM1_CH2N/TIM3_CH3/TIM8_CH2N)
- net HO_A: now also TP?.1
- net HO_B: now also TP?.1
- net HO_C: now also TP?.1
- net LI_A: now also U?.14 (PA0/ADC1_IN0/SYS_WKUP1/TIM2_CH1/TIM2_ETR/TIM5_CH1/TIM8_ETR/UART4_TX/USART2_CTS)
- net LI_B: now also U?.15 (PA1/ADC1_IN1/I2S4_SD/QUADSPI_BK1_IO3/SPI4_MOSI/TIM2_CH2/TIM5_CH2/UART4_RX/USART2_RTS)
- net LI_C: now also U?.16 (PA2/ADC1_IN2/FSMC_D4/FSMC_DA4/I2S_CKIN/TIM2_CH3/TIM5_CH3/TIM9_CH1/USART2_TX)
- net Sternpunkt_virtuell: now also TP?.1
- net Hochlauf: now reaches Q?.1 (G)
- net Hochlauf: now also U?.55 (PB3/CAN3_RX/FMPI2C1_SDA/I2C2_SDA/I2S1_CK/I2S3_CK/SAI1_SD_A/SPI1_SCK/SPI3_SCK/SYS_JTDO-SWO/TIM2_CH2/UART7_RX/USART1_RX)
- net elekKomm: now reaches Q?.1 (G)
- net elekKomm: now also U?.56 (PB4/CAN3_TX/I2C3_SDA/I2S3_ext_SD/SAI1_SCK_A/SDIO_D0/SPI1_MISO/SPI3_MISO/SYS_JTRST/TIM3_CH1/UART7_TX)
- new net: C?.2, U?.13 (VDDA)
- new net: C?.2, U?.19 (VDD)
- new net: C?.2, U?.32 (VDD)
- new net: C?.2, U?.48 (VDD)
- new net: C?.2, U?.64 (VDD)
- new net: C?.2, U?.30 (VCAP_1)
- new net: C?.2, U?.5 (PH0-OSC_IN/RCC_OSC_IN), Y?.1
- new net: C?.2, U?.6 (PH1-OSC_OUT/RCC_OSC_OUT), Y?.2
- new net D+: U?.45 (PA12/CAN1_TX/DFSDM2_DATIN5/SPI2_MISO/SPI5_MISO/TIM1_ETR/UART4_TX/USART1_RTS/USART6_RX/USB_OTG_FS_DP)
- new net D-: U?.44 (PA11/ADC1_EXTI11/CAN1_RX/DFSDM2_CKIN5/I2S2_WS/SPI2_NSS/SPI4_MISO/TIM1_CH4/UART4_RX/USART1_CTS/USART6_TX/USB_OTG_FS_DM)
- new net DAC1: U?.20 (PA4/ADC1_IN4/DAC_OUT1/DFSDM1_DATIN1/FSMC_D6/FSMC_DA6/I2S1_WS/I2S3_WS/SPI1_NSS/SPI3_NSS/USART2_CK)
- new net DAC2: U?.21 (PA5/ADC1_IN5/DAC_OUT2/DFSDM1_CKIN1/FSMC_D7/FSMC_DA7/I2S1_CK/SPI1_SCK/TIM2_CH1/TIM2_ETR/TIM8_CH1N)
- new net NRST: R?.2, SW?.1, U?.7 (NRST)
- new net SWCLK: U?.49 (PA14/SYS_JTCK-SWCLK)
- new net SWDIO: U?.46 (PA13/SYS_JTMS-SWDIO)
- new net SYSCLK_OUT: U?.40 (PC9/DAC_EXTI9/DFSDM2_DATIN3/I2C3_SDA/I2S_CKIN/QUADSPI_BK1_IO0/RCC_MCO_2/SDIO_D1/TIM3_CH4/TIM8_CH4)
Other:
- note added: "Motoranschluss"

Commit message: Netlist
Parts:
- added D4: USBLC6-2SC6Y, TO_SOT_Packages_SMD:SOT-23-6, symbol USBLC6-2SC6Y
- added J4: Conn_01x04, Connectors_JST:JST_EH_B04B-EH-A_04x2.50mm_Straight, symbol Conn_01x04
- added J5: USB_OTG, Connectors_USB:USB_Micro-B_Molex-105017-0001, symbol USB_OTG
- added R12, R14: 27, Resistors_SMD:R_0603, symbol R
- added R17: 3, Resistors_SMD:R_0603, symbol R
- added R42: 1k, Resistors_SMD:R_0603, symbol R
- added R8: 1,5k, Resistors_SMD:R_0603, symbol R
- added SW2: SW_Push, kicadBibs:Switch, symbol SW_Push
- added TP11, TP14, TP15, TP7, TP9: TEST, Pin_Headers:Pin_Header_Straight_1x01_Pitch1.00mm, symbol TEST
- R16: renamed from R?; footprint (none) -> Resistors_SMD:R_0603
- SW1: renamed from SW?; footprint (none) -> kicadBibs:Switch
- U12: renamed from U?; footprint LQFP64 -> Housings_QFP:LQFP-64_10x10mm_Pitch0.5mm
- Y1: renamed from Y?; footprint (none) -> kicadBibs:FQ5032A
- gave numbers to parts that had none: 116
Connections:
- net +3V3: now also J4.1 (Pin_1), R8.2, SW2.1
- net A_conn: now also U12.8 (PC0/ADC1_IN10/DFSDM2_CKIN4/LPTIM1_IN1/SAI1_MCLK_B/SYS_WKUP2)
- net B_conn: now also U12.9 (PC1/ADC1_IN11/DFSDM2_DATIN4/LPTIM1_OUT/SAI1_SD_B/SYS_WKUP3)
- net Bemf_A: now also U12.41 (PA8/CAN3_RX/DFSDM1_CKOUT/I2C3_SCL/RCC_MCO_1/SDIO_D1/TIM1_CH1/UART7_RX/USART1_CK/USB_OTG_FS_SOF); no longer U12.41 (PA8/CAN3_RX/DFSDM1_CKOUT/I2C3_SCL/RCC_MCO_1/SDIO_D1/TIM1_CH1/UART7_RX/USART1_CK/USB_OTG_FS_SOF)
- net Bemf_B: now also U12.42 (PA9/DAC_EXTI9/DFSDM2_CKIN3/I2C3_SMBA/I2S2_CK/SDIO_D2/SPI2_SCK/TIM1_CH2/USART1_TX/USB_OTG_FS_VBUS); no longer U12.42 (PA9/DAC_EXTI9/DFSDM2_CKIN3/I2C3_SMBA/I2S2_CK/SDIO_D2/SPI2_SCK/TIM1_CH2/USART1_TX/USB_OTG_FS_VBUS)
- net Bemf_C: now also U12.43 (PA10/DFSDM2_DATIN3/I2S2_SD/I2S5_SD/SPI2_MOSI/SPI5_MOSI/TIM1_CH3/USART1_RX/USB_OTG_FS_ID); no longer U12.43 (PA10/DFSDM2_DATIN3/I2S2_SD/I2S5_SD/SPI2_MOSI/SPI5_MOSI/TIM1_CH3/USART1_RX/USB_OTG_FS_ID)
- net C: now also U12.10 (PC2/ADC1_IN12/DFSDM1_CKOUT/DFSDM2_DATIN7/FSMC_NWE/I2S2_ext_SD/LPTIM1_IN2/SAI1_SCK_B/SPI2_MISO)
- net Curr_mcu_A: now also U12.24 (PC4/ADC1_IN14/DFSDM2_CKIN2/FSMC_NE4/I2S1_MCK/QUADSPI_BK2_IO2); no longer U12.8 (PC0/ADC1_IN10/DFSDM2_CKIN4/LPTIM1_IN1/SAI1_MCLK_B/SYS_WKUP2)
- net Curr_mcu_B: now also U12.25 (PC5/ADC1_IN15/DFSDM2_DATIN2/FMPI2C1_SMBA/FSMC_NOE/QUADSPI_BK2_IO3/USART3_RX); no longer U12.9 (PC1/ADC1_IN11/DFSDM2_DATIN4/LPTIM1_OUT/SAI1_SD_B/SYS_WKUP3)
- net D+: now also U12.45 (PA12/CAN1_TX/DFSDM2_DATIN5/SPI2_MISO/SPI5_MISO/TIM1_ETR/UART4_TX/USART1_RTS/USART6_RX/USB_OTG_FS_DP), D4.6 (IO1); no longer U12.45 (PA12/CAN1_TX/DFSDM2_DATIN5/SPI2_MISO/SPI5_MISO/TIM1_ETR/UART4_TX/USART1_RTS/USART6_RX/USB_OTG_FS_DP)
- net D-: now also U12.44 (PA11/ADC1_EXTI11/CAN1_RX/DFSDM2_CKIN5/I2S2_WS/SPI2_NSS/SPI4_MISO/TIM1_CH4/UART4_RX/USART1_CTS/USART6_TX/USB_OTG_FS_DM), D4.4 (IO2); no longer U12.44 (PA11/ADC1_EXTI11/CAN1_RX/DFSDM2_CKIN5/I2S2_WS/SPI2_NSS/SPI4_MISO/TIM1_CH4/UART4_RX/USART1_CTS/USART6_TX/USB_OTG_FS_DM)
- net DAC1: now also U12.20 (PA4/ADC1_IN4/DAC_OUT1/DFSDM1_DATIN1/FSMC_D6/FSMC_DA6/I2S1_WS/I2S3_WS/SPI1_NSS/SPI3_NSS/USART2_CK), TP14.1; no longer U12.20 (PA4/ADC1_IN4/DAC_OUT1/DFSDM1_DATIN1/FSMC_D6/FSMC_DA6/I2S1_WS/I2S3_WS/SPI1_NSS/SPI3_NSS/USART2_CK)
- net DAC2: now also U12.21 (PA5/ADC1_IN5/DAC_OUT2/DFSDM1_CKIN1/FSMC_D7/FSMC_DA7/I2S1_CK/SPI1_SCK/TIM2_CH1/TIM2_ETR/TIM8_CH1N), TP15.1; no longer U12.21 (PA5/ADC1_IN5/DAC_OUT2/DFSDM1_CKIN1/FSMC_D7/FSMC_DA7/I2S1_CK/SPI1_SCK/TIM2_CH1/TIM2_ETR/TIM8_CH1N)
- net Freigabe_MCU: now also U12.57 (PB5/CAN2_RX/I2C1_SMBA/I2S1_SD/I2S3_SD/LPTIM1_IN1/SAI1_FS_A/SDIO_D3/SPI1_MOSI/SPI3_MOSI/TIM3_CH2/UART5_RX), U7.10; no longer U7.13
- net Freigabe_button: now also U7.9, R42.1, SW2.2; no longer U7.12
- net GNDREF: now also U12.12 (VSSA), U12.18 (VSS), U12.31 (VSS), U12.47 (VSS), U12.60 (BOOT0), U12.63 (VSS), D4.2 (GND), J4.4 (Pin_4), J5.5 (GND), R17.1, R42.2; no longer U12.12 (VSSA), U12.18 (VSS), U12.31 (VSS), U12.47 (VSS), U12.60 (BOOT0), U12.63 (VSS)
- net HI_A: now also U12.22 (PA6/ADC1_IN6/DFSDM2_CKIN1/I2S2_MCK/QUADSPI_BK2_IO0/SDIO_CMD/SPI1_MISO/TIM13_CH1/TIM1_BKIN/TIM3_CH1/TIM8_BKIN); no longer U12.22 (PA6/ADC1_IN6/DFSDM2_CKIN1/I2S2_MCK/QUADSPI_BK2_IO0/SDIO_CMD/SPI1_MISO/TIM13_CH1/TIM1_BKIN/TIM3_CH1/TIM8_BKIN)
- net HI_B: now also U12.23 (PA7/ADC1_IN7/DFSDM2_DATIN1/I2S1_SD/QUADSPI_BK2_IO1/SPI1_MOSI/TIM14_CH1/TIM1_CH1N/TIM3_CH2/TIM8_CH1N); no longer U12.23 (PA7/ADC1_IN7/DFSDM2_DATIN1/I2S1_SD/QUADSPI_BK2_IO1/SPI1_MOSI/TIM14_CH1/TIM1_CH1N/TIM3_CH2/TIM8_CH1N)
- net HI_C: now also U12.26 (PB0/ADC1_IN8/I2S5_CK/SPI5_SCK/TIM1_CH2N/TIM3_CH3/TIM8_CH2N); no longer U12.26 (PB0/ADC1_IN8/I2S5_CK/SPI5_SCK/TIM1_CH2N/TIM3_CH3/TIM8_CH2N)
- net Hochlauf: now also U12.55 (PB3/CAN3_RX/FMPI2C1_SDA/I2C2_SDA/I2S1_CK/I2S3_CK/SAI1_SD_A/SPI1_SCK/SPI3_SCK/SYS_JTDO-SWO/TIM2_CH2/UART7_RX/USART1_RX); no longer U12.55 (PB3/CAN3_RX/FMPI2C1_SDA/I2C2_SDA/I2S1_CK/I2S3_CK/SAI1_SD_A/SPI1_SCK/SPI3_SCK/SYS_JTDO-SWO/TIM2_CH2/UART7_RX/USART1_RX)
- net LI_A: now also U12.14 (PA0/ADC1_IN0/SYS_WKUP1/TIM2_CH1/TIM2_ETR/TIM5_CH1/TIM8_ETR/UART4_TX/USART2_CTS); no longer U12.14 (PA0/ADC1_IN0/SYS_WKUP1/TIM2_CH1/TIM2_ETR/TIM5_CH1/TIM8_ETR/UART4_TX/USART2_CTS)
- net LI_B: now also U12.15 (PA1/ADC1_IN1/I2S4_SD/QUADSPI_BK1_IO3/SPI4_MOSI/TIM2_CH2/TIM5_CH2/UART4_RX/USART2_RTS); no longer U12.15 (PA1/ADC1_IN1/I2S4_SD/QUADSPI_BK1_IO3/SPI4_MOSI/TIM2_CH2/TIM5_CH2/UART4_RX/USART2_RTS)
- net LI_C: now also U12.16 (PA2/ADC1_IN2/FSMC_D4/FSMC_DA4/I2S_CKIN/TIM2_CH3/TIM5_CH3/TIM9_CH1/USART2_TX); no longer U12.16 (PA2/ADC1_IN2/FSMC_D4/FSMC_DA4/I2S_CKIN/TIM2_CH3/TIM5_CH3/TIM9_CH1/USART2_TX)
- net LO_A: now also TP7.1
- net LO_B: now also TP9.1
- net LO_C: now also TP11.1
- net NRST: now also U12.7 (NRST); no longer U12.7 (NRST)
- net OR1: now also U7.1, U7.6; no longer U7.3, U7.9
- net OR2: now also U7.11, U7.2; no longer U7.10, U7.6
- net SWCLK: now also U12.49 (PA14/SYS_JTCK-SWCLK), J4.3 (Pin_3); no longer U12.49 (PA14/SYS_JTCK-SWCLK)
- net SWDIO: now also U12.46 (PA13/SYS_JTMS-SWDIO); no longer U12.46 (PA13/SYS_JTMS-SWDIO)
- net SYSCLK_OUT: now also U12.40 (PC9/DAC_EXTI9/DFSDM2_DATIN3/I2C3_SDA/I2S_CKIN/QUADSPI_BK1_IO0/RCC_MCO_2/SDIO_D1/TIM3_CH4/TIM8_CH4); no longer U12.40 (PC9/DAC_EXTI9/DFSDM2_DATIN3/I2C3_SDA/I2S_CKIN/QUADSPI_BK1_IO0/RCC_MCO_2/SDIO_D1/TIM3_CH4/TIM8_CH4)
- net Sternpunkt_virtuell: now also U12.11 (PC3/ADC1_IN13/DFSDM2_CKIN7/FSMC_A0/I2S2_SD/LPTIM1_ETR/SAI1_FS_B/SPI2_MOSI)
- net Stop: now also U7.3; no longer U7.8
- net elekKomm: now also U12.56 (PB4/CAN3_TX/I2C3_SDA/I2S3_ext_SD/SAI1_SCK_A/SDIO_D0/SPI1_MISO/SPI3_MISO/SYS_JTRST/TIM3_CH1/UART7_TX); no longer U12.56 (PB4/CAN3_TX/I2C3_SDA/I2S3_ext_SD/SAI1_SCK_A/SDIO_D0/SPI1_MISO/SPI3_MISO/SYS_JTRST/TIM3_CH1/UART7_TX)
- net at R27.2: now also U7.8; no longer U7.11
- net at R22.2, U11.2: now also U7.4; no longer U7.1
- net at R28.2, U11.1: now also U7.5; no longer U7.2
- net at R32.2, U11.14: now also U7.12; no longer U7.4
- net at R40.2, U11.13: now also U7.13; no longer U7.5
- net at C26.2: now also U12.13 (VDDA); no longer U12.13 (VDDA)
- net at C18.2: now also U12.19 (VDD); no longer U12.19 (VDD)
- net at C20.2: now also U12.32 (VDD); no longer U12.32 (VDD)
- net at C22.2: now also U12.48 (VDD); no longer U12.48 (VDD)
- net at C24.2: now also U12.64 (VDD); no longer U12.64 (VDD)
- net at C25.2: now also U12.30 (VCAP_1); no longer U12.30 (VCAP_1)
- new net: J5.2 (D-), R14.2
- new net: J5.3 (D+), R12.2
- new net: J5.6 (Shield), R17.2
- new net: D4.1 (IO1), R12.1, R8.1
- new net: D4.3 (IO2), R14.1
- new net SWIO: J4.2 (Pin_2)
Other:
- note added: "Back-EMF Detektoren"
- note added: "Testpunkte"
- moved on the sheet: R41, SW1

Commit message: Schematic fertig
Parts:
- C19: footprint (none) -> Capacitors_SMD:C_0603
- D10, D8, D9: footprint (none) -> LEDs:LED_0805
- D6, D7: footprint (none) -> LEDs:LED_0805_HandSoldering
- U12: footprint LQFP64 -> Housings_QFP:LQFP-64_10x10mm_Pitch0.5mm
- U7: footprint (none) -> Housings_SSOP:TSSOP-14_4.4x5mm_Pitch0.65mm
- U8: footprint (none) -> Housings_SSOP:TSSOP-8_3x3mm_Pitch0.65mm
Changed lines of the file:
@@
 F 0 "U8" H 8950 8050 60  0000 C CNN
 F 1 "74LVC2G02" H 8950 7950 60  0000 C CNN
-F 2 "" H 8950 8150 60  0001 C CNN
+F 2 "Housings_SSOP:TSSOP-8_3x3mm_Pitch0.65mm" H 8950 8150 60  0001 C CNN
 F 3 "" H 8950 8150 60  0001 C CNN
 	2    8950 8150
@@
 F 0 "C19" H 8475 8350 50  0000 L CNN
 F 1 "100n" H 8475 8150 50  0000 L CNN
-F 2 "" H 8488 8100 50  0001 C CNN
+F 2 "Capacitors_SMD:C_0603" H 8488 8100 50  0001 C CNN
 F 3 "" H 8450 8250 50  0001 C CNN
 	1    8450 8250
@@
 F 0 "U7" H 4100 7050 60  0000 C CNN
 F 1 "74HC32D" H 4200 6950 60  0000 C CNN
-F 2 "" H 3850 7150 60  0001 C CNN
+F 2 "Housings_SSOP:TSSOP-14_4.4x5mm_Pitch0.65mm" H 3850 7150 60  0001 C CNN
 F 3 "" H 3850 7150 60  0001 C CNN
 	2    3850 7150
@@
 F 0 "U7" H 4050 11250 60  0000 C CNN
 F 1 "74HC32D" H 4000 11150 60  0000 C CNN
-F 2 "" H 4000 11350 60  0001 C CNN
+F 2 "Housings_SSOP:TSSOP-14_4.4x5mm_Pitch0.65mm" H 4000 11350 60  0001 C CNN
 F 3 "" H 4000 11350 60  0001 C CNN
 	4    4000 11350
@@
 F 0 "U7" H 7000 6800 60  0000 C CNN
 F 1 "74HC32D" H 6950 6700 60  0000 C CNN
-F 2 "" H 6950 6900 60  0001 C CNN
+F 2 "Housings_SSOP:TSSOP-14_4.4x5mm_Pitch0.65mm" H 6950 6900 60  0001 C CNN
 F 3 "" H 6950 6900 60  0001 C CNN
 	1    6950 6900
@@
 F 0 "U7" H 5900 8250 60  0000 C CNN
 F 1 "74HC32D" H 5850 8150 60  0000 C CNN
-F 2 "" H 5850 8350 60  0001 C CNN
+F 2 "Housings_SSOP:TSSOP-14_4.4x5mm_Pitch0.65mm" H 5850 8350 60  0001 C CNN
 F 3 "" H 5850 8350 60  0001 C CNN
 	3    5850 8350
@@
 F 0 "D7" H 8150 12100 50  0000 C CNN
 F 1 "LED_ALT" H 8150 11900 50  0000 C CNN
-F 2 "" H 8150 12000 50  0001 C CNN
+F 2 "LEDs:LED_0805_HandSoldering" H 8150 12000 50  0001 C CNN
 F 3 "" H 8150 12000 50  0001 C CNN
 	1    8150 12000
@@
 F 0 "D6" H 7350 12100 50  0000 C CNN
 F 1 "LED_ALT" H 7350 11900 50  0000 C CNN
-F 2 "" H 7350 12000 50  0001 C CNN
+F 2 "LEDs:LED_0805_HandSoldering" H 7350 12000 50  0001 C CNN
 F 3 "" H 7350 12000 50  0001 C CNN
 	1    7350 12000
@@
 F 0 "D8" H 8900 12100 50  0000 C CNN
 F 1 "LED_ALT" H 8900 11900 50  0000 C CNN
-F 2 "" H 8900 12000 50  0001 C CNN
+F 2 "LEDs:LED_0805" H 8900 12000 50  0001 C CNN
 F 3 "" H 8900 12000 50  0001 C CNN
 	1    8900 12000
@@
 F 0 "D9" H 9650 12100 50  0000 C CNN
 F 1 "LED_ALT" H 9650 11900 50  0000 C CNN
-F 2 "" H 9650 12000 50  0001 C CNN
+F 2 "LEDs:LED_0805" H 9650 12000 50  0001 C CNN
 F 3 "" H 9650 12000 50  0001 C CNN
 	1    9650 12000
@@
 F 0 "D10" H 10300 12100 50  0000 C CNN
 F 1 "LED_ALT" H 10300 11900 50  0000 C CNN
-F 2 "" H 10300 12000 50  0001 C CNN
+F 2 "LEDs:LED_0805" H 10300 12000 50  0001 C CNN
 F 3 "" H 10300 12000 50  0001 C CNN
 	1    10300 12000
@@
 F 0 "U12" H 13850 11950 50  0000 C CNN
 F 1 "STM32F413R(G-H)Tx_u" H 13850 11750 50  0000 C CNN
-F 2 "LQFP64" H 13850 11650 50  0000 C CIN
+F 2 "Housings_QFP:LQFP-64_10x10mm_Pitch0.5mm" H 13850 11650 50  0000 C CIN
 F 3 "" H 13850 11850 50  0000 C CNN
 	2    13850 11850
@@
 F 0 "U12" H 13700 10100 50  0000 C CNN
 F 1 "STM32F413R(G-H)Tx_u" H 13700 9900 50  0000 C CNN
-F 2 "LQFP64" H 13700 9800 50  0000 C CIN
+F 2 "Housings_QFP:LQFP-64_10x10mm_Pitch0.5mm" H 13700 9800 50  0000 C CIN
 F 3 "" H 13700 10000 50  0000 C CNN
 	3    13700 10000
@@
 F 0 "U12" H 16650 8150 50  0000 C CNN
 F 1 "STM32F413R(G-H)Tx_u" H 16650 7950 50  0000 C CNN
-F 2 "LQFP64" H 16650 7850 50  0000 C CIN
+F 2 "Housings_QFP:LQFP-64_10x10mm_Pitch0.5mm" H 16650 7850 50  0000 C CIN
 F 3 "" H 16650 8050 50  0000 C CNN
 	4    16650 8050
@@
 F 0 "U12" H 16350 8650 50  0000 C CNN
 F 1 "STM32F413R(G-H)Tx_u" H 16350 8450 50  0000 C CNN
-F 2 "LQFP64" H 16350 8350 50  0000 C CIN
+F 2 "Housings_QFP:LQFP-64_10x10mm_Pitch0.5mm" H 16350 8350 50  0000 C CIN
 F 3 "" H 16350 8550 50  0000 C CNN
 	5    16350 8550
@@
 F 0 "U12" H 13750 13850 50  0000 C CNN
 F 1 "STM32F413R(G-H)Tx_u" H 13750 13650 50  0000 C CNN
-F 2 "LQFP64" H 13750 13550 50  0000 C CIN
+F 2 "Housings_QFP:LQFP-64_10x10mm_Pitch0.5mm" H 13750 13550 50  0000 C CIN
 F 3 "" H 13750 13750 50  0000 C CNN
 	1    13750 13750
@@
 F 0 "U12" H 13050 8600 50  0000 C CNN
 F 1 "STM32F413R(G-H)Tx_u" H 13050 8400 50  0000 C CNN
-F 2 "LQFP64" H 13050 8300 50  0000 C CIN
+F 2 "Housings_QFP:LQFP-64_10x10mm_Pitch0.5mm" H 13050 8300 50  0000 C CIN
 F 3 "" H 13050 8500 50  0000 C CNN
 	7    13050 8500
@@
 F 0 "U12" H 11450 8600 50  0000 C CNN
 F 1 "STM32F413R(G-H)Tx_u" H 11450 8400 50  0000 C CNN
-F 2 "LQFP64" H 11450 8300 50  0000 C CIN
+F 2 "Housings_QFP:LQFP-64_10x10mm_Pitch0.5mm" H 11450 8300 50  0000 C CIN
 F 3 "" H 11450 8500 50  0000 C CNN
 	8    11450 8500
