File: Hardware/Elektrische_Komm.sch (KiCad schematic (older format))
At the start: 133 parts, among them J1 Conn_01x01, J2 Conn_01x01, J3 Conn_01x01, J4 Conn_01x04, J5 USB_OTG, Q1 BSZ014NE2LS5IF, Q10 BSR202NL6327HTSA1, Q11 BSR202NL6327HTSA1, Q12 BSR202NL6327HTSA1, Q13 BSR202NL6327HTSA1, Q14 BSR202NL6327HTSA1, Q2 BSZ014NE2LS5IF, Q3 BSZ014NE2LS5IF, Q4 BSZ014NE2LS5IF, Q5 BSZ014NE2LS5IF, Q6 BSZ014NE2LS5IF, Q7 BSR202NL6327HTSA1, Q8 BSR202NL6327HTSA1, Q9 BSR202NL6327HTSA1, SW1 SW_Push, SW2 SW_Push, U1 TS374IDT, U10 TPS561201, U11 LVM339IDT, U12 STM32F413R(G-H)Tx_u, U2 UCC27710, U3 ACS723LLCTR, U4 UCC27710, U5 ACS723LLCTR, U6 UCC27710, U7 74HC32D, U8 74LVC2G02, U9 LDK715M50R, Y1 10MHz

Commit message: Layout
Parts:
- added C50, C51: 100n, Capacitors_SMD:C_0603, symbol C
- added TP18: TEST, Pin_Headers:Pin_Header_Straight_1x01_Pitch1.00mm, symbol TEST
- U11: footprint (none) -> Housings_SOIC:SOIC-14_3.9x8.7mm_Pitch1.27mm
- renumbered TP18 to TP19, TP19 to TP20, TP20 to TP21
Connections:
- net SWIO is gone; now on net SWDIO: J4.2 (Pin_2)
- net +3V3: now also C18.2, C20.2, C22.2, C24.2, C26.2, U12.13 (VDDA), U12.19 (VDD), U12.32 (VDD), U12.48 (VDD), U12.64 (VDD)
- net +5V: now also C50.1, C51.1
- net A_conn: now also U12.8 (PC0/ADC1_IN10/DFSDM2_CKIN4/LPTIM1_IN1/SAI1_MCLK_B/SYS_WKUP2); no longer U12.8 (PC0/ADC1_IN10/DFSDM2_CKIN4/LPTIM1_IN1/SAI1_MCLK_B/SYS_WKUP2)
- net B_conn: now also U12.9 (PC1/ADC1_IN11/DFSDM2_DATIN4/LPTIM1_OUT/SAI1_SD_B/SYS_WKUP3); no longer U12.9 (PC1/ADC1_IN11/DFSDM2_DATIN4/LPTIM1_OUT/SAI1_SD_B/SYS_WKUP3)
- net Bemf_A: now also U12.41 (PA8/CAN3_RX/DFSDM1_CKOUT/I2C3_SCL/RCC_MCO_1/SDIO_D1/TIM1_CH1/UART7_RX/USART1_CK/USB_OTG_FS_SOF); no longer U12.41 (PA8/CAN3_RX/DFSDM1_CKOUT/I2C3_SCL/RCC_MCO_1/SDIO_D1/TIM1_CH1/UART7_RX/USART1_CK/USB_OTG_FS_SOF)
- net Bemf_B: now also U12.42 (PA9/DAC_EXTI9/DFSDM2_CKIN3/I2C3_SMBA/I2S2_CK/SDIO_D2/SPI2_SCK/TIM1_CH2/USART1_TX/USB_OTG_FS_VBUS); no longer U12.42 (PA9/DAC_EXTI9/DFSDM2_CKIN3/I2C3_SMBA/I2S2_CK/SDIO_D2/SPI2_SCK/TIM1_CH2/USART1_TX/USB_OTG_FS_VBUS)
- net Bemf_C: now also U12.43 (PA10/DFSDM2_DATIN3/I2S2_SD/I2S5_SD/SPI2_MOSI/SPI5_MOSI/TIM1_CH3/USART1_RX/USB_OTG_FS_ID); no longer U12.43 (PA10/DFSDM2_DATIN3/I2S2_SD/I2S5_SD/SPI2_MOSI/SPI5_MOSI/TIM1_CH3/USART1_RX/USB_OTG_FS_ID)
- net C: now also U12.10 (PC2/ADC1_IN12/DFSDM1_CKOUT/DFSDM2_DATIN7/FSMC_NWE/I2S2_ext_SD/LPTIM1_IN2/SAI1_SCK_B/SPI2_MISO); no longer U12.10 (PC2/ADC1_IN12/DFSDM1_CKOUT/DFSDM2_DATIN7/FSMC_NWE/I2S2_ext_SD/LPTIM1_IN2/SAI1_SCK_B/SPI2_MISO)
- net Curr_mcu_A: now also U12.24 (PC4/ADC1_IN14/DFSDM2_CKIN2/FSMC_NE4/I2S1_MCK/QUADSPI_BK2_IO2); no longer U12.24 (PC4/ADC1_IN14/DFSDM2_CKIN2/FSMC_NE4/I2S1_MCK/QUADSPI_BK2_IO2)
- net Curr_mcu_B: now also U12.25 (PC5/ADC1_IN15/DFSDM2_DATIN2/FMPI2C1_SMBA/FSMC_NOE/QUADSPI_BK2_IO3/USART3_RX); no longer U12.25 (PC5/ADC1_IN15/DFSDM2_DATIN2/FMPI2C1_SMBA/FSMC_NOE/QUADSPI_BK2_IO3/USART3_RX)
- net D+: now also D4.4 (IO2), U12.45 (PA12/CAN1_TX/DFSDM2_DATIN5/SPI2_MISO/SPI5_MISO/TIM1_ETR/UART4_TX/USART1_RTS/USART6_RX/USB_OTG_FS_DP); no longer D4.6 (IO1), U12.45 (PA12/CAN1_TX/DFSDM2_DATIN5/SPI2_MISO/SPI5_MISO/TIM1_ETR/UART4_TX/USART1_RTS/USART6_RX/USB_OTG_FS_DP)
- net D-: now also D4.6 (IO1), U12.44 (PA11/ADC1_EXTI11/CAN1_RX/DFSDM2_CKIN5/I2S2_WS/SPI2_NSS/SPI4_MISO/TIM1_CH4/UART4_RX/USART1_CTS/USART6_TX/USB_OTG_FS_DM); no longer D4.4 (IO2), U12.44 (PA11/ADC1_EXTI11/CAN1_RX/DFSDM2_CKIN5/I2S2_WS/SPI2_NSS/SPI4_MISO/TIM1_CH4/UART4_RX/USART1_CTS/USART6_TX/USB_OTG_FS_DM)
- net DAC1: now also U12.20 (PA4/ADC1_IN4/DAC_OUT1/DFSDM1_DATIN1/FSMC_D6/FSMC_DA6/I2S1_WS/I2S3_WS/SPI1_NSS/SPI3_NSS/USART2_CK); no longer U12.20 (PA4/ADC1_IN4/DAC_OUT1/DFSDM1_DATIN1/FSMC_D6/FSMC_DA6/I2S1_WS/I2S3_WS/SPI1_NSS/SPI3_NSS/USART2_CK)
- net DAC2: now also U12.21 (PA5/ADC1_IN5/DAC_OUT2/DFSDM1_CKIN1/FSMC_D7/FSMC_DA7/I2S1_CK/SPI1_SCK/TIM2_CH1/TIM2_ETR/TIM8_CH1N); no longer U12.21 (PA5/ADC1_IN5/DAC_OUT2/DFSDM1_CKIN1/FSMC_D7/FSMC_DA7/I2S1_CK/SPI1_SCK/TIM2_CH1/TIM2_ETR/TIM8_CH1N)
- net Freigabe_MCU: now also U12.57 (PB5/CAN2_RX/I2C1_SMBA/I2S1_SD/I2S3_SD/LPTIM1_IN1/SAI1_FS_A/SDIO_D3/SPI1_MOSI/SPI3_MOSI/TIM3_CH2/UART5_RX); no longer U12.57 (PB5/CAN2_RX/I2C1_SMBA/I2S1_SD/I2S3_SD/LPTIM1_IN1/SAI1_FS_A/SDIO_D3/SPI1_MOSI/SPI3_MOSI/TIM3_CH2/UART5_RX)
- net GNDREF: now also U12.12 (VSSA), U12.18 (VSS), U12.31 (VSS), U12.47 (VSS), U12.60 (BOOT0), U12.63 (VSS), C50.2, C51.2; no longer U12.12 (VSSA), U12.18 (VSS), U12.31 (VSS), U12.47 (VSS), U12.60 (BOOT0), U12.63 (VSS)
- net HI_A: now also U12.22 (PA6/ADC1_IN6/DFSDM2_CKIN1/I2S2_MCK/QUADSPI_BK2_IO0/SDIO_CMD/SPI1_MISO/TIM13_CH1/TIM1_BKIN/TIM3_CH1/TIM8_BKIN); no longer U12.22 (PA6/ADC1_IN6/DFSDM2_CKIN1/I2S2_MCK/QUADSPI_BK2_IO0/SDIO_CMD/SPI1_MISO/TIM13_CH1/TIM1_BKIN/TIM3_CH1/TIM8_BKIN)
- net HI_B: now also U12.23 (PA7/ADC1_IN7/DFSDM2_DATIN1/I2S1_SD/QUADSPI_BK2_IO1/SPI1_MOSI/TIM14_CH1/TIM1_CH1N/TIM3_CH2/TIM8_CH1N); no longer U12.23 (PA7/ADC1_IN7/DFSDM2_DATIN1/I2S1_SD/QUADSPI_BK2_IO1/SPI1_MOSI/TIM14_CH1/TIM1_CH1N/TIM3_CH2/TIM8_CH1N)
- net HI_C: now also U12.26 (PB0/ADC1_IN8/I2S5_CK/SPI5_SCK/TIM1_CH2N/TIM3_CH3/TIM8_CH2N); no longer U12.26 (PB0/ADC1_IN8/I2S5_CK/SPI5_SCK/TIM1_CH2N/TIM3_CH3/TIM8_CH2N)
- net Hochlauf: now also U12.55 (PB3/CAN3_RX/FMPI2C1_SDA/I2C2_SDA/I2S1_CK/I2S3_CK/SAI1_SD_A/SPI1_SCK/SPI3_SCK/SYS_JTDO-SWO/TIM2_CH2/UART7_RX/USART1_RX); no longer U12.55 (PB3/CAN3_RX/FMPI2C1_SDA/I2C2_SDA/I2S1_CK/I2S3_CK/SAI1_SD_A/SPI1_SCK/SPI3_SCK/SYS_JTDO-SWO/TIM2_CH2/UART7_RX/USART1_RX)
- net LI_A: now also U12.14 (PA0/ADC1_IN0/SYS_WKUP1/TIM2_CH1/TIM2_ETR/TIM5_CH1/TIM8_ETR/UART4_TX/USART2_CTS); no longer U12.14 (PA0/ADC1_IN0/SYS_WKUP1/TIM2_CH1/TIM2_ETR/TIM5_CH1/TIM8_ETR/UART4_TX/USART2_CTS)
- net LI_B: now also U12.15 (PA1/ADC1_IN1/I2S4_SD/QUADSPI_BK1_IO3/SPI4_MOSI/TIM2_CH2/TIM5_CH2/UART4_RX/USART2_RTS); no longer U12.15 (PA1/ADC1_IN1/I2S4_SD/QUADSPI_BK1_IO3/SPI4_MOSI/TIM2_CH2/TIM5_CH2/UART4_RX/USART2_RTS)
- net LI_C: now also U12.16 (PA2/ADC1_IN2/FSMC_D4/FSMC_DA4/I2S_CKIN/TIM2_CH3/TIM5_CH3/TIM9_CH1/USART2_TX); no longer U12.16 (PA2/ADC1_IN2/FSMC_D4/FSMC_DA4/I2S_CKIN/TIM2_CH3/TIM5_CH3/TIM9_CH1/USART2_TX)
- net NRST: now also U12.7 (NRST); no longer U12.7 (NRST)
- net SWCLK: now also U12.49 (PA14/SYS_JTCK-SWCLK); no longer U12.49 (PA14/SYS_JTCK-SWCLK)
- net SWDIO: now also U12.46 (PA13/SYS_JTMS-SWDIO); no longer U12.46 (PA13/SYS_JTMS-SWDIO)
- net SYSCLK_OUT: now also U12.40 (PC9/DAC_EXTI9/DFSDM2_DATIN3/I2C3_SDA/I2S_CKIN/QUADSPI_BK1_IO0/RCC_MCO_2/SDIO_D1/TIM3_CH4/TIM8_CH4), TP18.1; no longer U12.40 (PC9/DAC_EXTI9/DFSDM2_DATIN3/I2C3_SDA/I2S_CKIN/QUADSPI_BK1_IO0/RCC_MCO_2/SDIO_D1/TIM3_CH4/TIM8_CH4)
- net Sternpunkt_virtuell: now also U12.11 (PC3/ADC1_IN13/DFSDM2_CKIN7/FSMC_A0/I2S2_SD/LPTIM1_ETR/SAI1_FS_B/SPI2_MOSI); no longer U12.11 (PC3/ADC1_IN13/DFSDM2_CKIN7/FSMC_A0/I2S2_SD/LPTIM1_ETR/SAI1_FS_B/SPI2_MOSI)
- net elekKomm: now also U12.56 (PB4/CAN3_TX/I2C3_SDA/I2S3_ext_SD/SAI1_SCK_A/SDIO_D0/SPI1_MISO/SPI3_MISO/SYS_JTRST/TIM3_CH1/UART7_TX); no longer U12.56 (PB4/CAN3_TX/I2C3_SDA/I2S3_ext_SD/SAI1_SCK_A/SDIO_D0/SPI1_MISO/SPI3_MISO/SYS_JTRST/TIM3_CH1/UART7_TX)
- net at C25.2: now also U12.30 (VCAP_1); no longer U12.30 (VCAP_1)
- net at R12.1, R8.1: now also D4.3 (IO2); no longer D4.1 (IO1)
- net at R14.1: now also D4.1 (IO1); no longer D4.3 (IO2)
Changed lines of the file:
@@
 F 0 "U11" H 2050 7350 60  0000 C CNN
 F 1 "LVM339IDT" H 2150 7250 60  0000 C CNN
-F 2 "" H 2000 7200 60  0001 C CNN
+F 2 "Housings_SOIC:SOIC-14_3.9x8.7mm_Pitch1.27mm" H 2000 7200 60  0001 C CNN
 F 3 "" H 2000 7200 60  0001 C CNN
 	1    2000 7200
@@
 F 0 "U11" H 2000 8950 60  0000 C CNN
 F 1 "LVM339IDT" H 2000 8850 60  0000 C CNN
-F 2 "" H 2000 9000 60  0001 C CNN
+F 2 "Housings_SOIC:SOIC-14_3.9x8.7mm_Pitch1.27mm" H 2000 9000 60  0001 C CNN
 F 3 "" H 2000 9000 60  0001 C CNN
 	2    2000 9000
@@
 F 0 "U11" H 2000 10750 60  0000 C CNN
 F 1 "LVM339IDT" H 2000 10650 60  0000 C CNN
-F 2 "" H 2000 10800 60  0001 C CNN
+F 2 "Housings_SOIC:SOIC-14_3.9x8.7mm_Pitch1.27mm" H 2000 10800 60  0001 C CNN
 F 3 "" H 2000 10800 60  0001 C CNN
 	3    2000 10800
@@
 F 0 "U11" H 2000 12550 60  0000 C CNN
 F 1 "LVM339IDT" H 2000 12450 60  0000 C CNN
-F 2 "" H 2000 12600 60  0001 C CNN
+F 2 "Housings_SOIC:SOIC-14_3.9x8.7mm_Pitch1.27mm" H 2000 12600 60  0001 C CNN
 F 3 "" H 2000 12600 60  0001 C CNN
 	4    2000 12600
@@
 $EndComp
 $Comp
-L TEST TP18
+L TEST TP19
 U 1 1 5AFCA395
 P 1100 15400
-F 0 "TP18" H 1100 15700 50  0000 C BNN
+F 0 "TP19" H 1100 15700 50  0000 C BNN
 F 1 "TEST" H 1100 15650 50  0000 C CNN
 F 2 "Pin_Headers:Pin_Header_Straight_1x01_Pitch1.00mm" H 1100 15400 50  0001 C CNN
@@
 $EndComp
 $Comp
-L TEST TP19
+L TEST TP20
 U 1 1 5AFCA4F0
 P 1100 15600
-F 0 "TP19" H 1100 15900 50  0000 C BNN
+F 0 "TP20" H 1100 15900 50  0000 C BNN
 F 1 "TEST" H 1100 15850 50  0000 C CNN
 F 2 "Pin_Headers:Pin_Header_Straight_1x01_Pitch1.00mm" H 1100 15600 50  0001 C CNN
@@
 $EndComp
 $Comp
-L TEST TP20
+L TEST TP21
 U 1 1 5AFCA64E
 P 1100 15850
-F 0 "TP20" H 1100 16150 50  0000 C BNN
+F 0 "TP21" H 1100 16150 50  0000 C BNN
 F 1 "TEST" H 1100 16100 50  0000 C CNN
 F 2 "Pin_Headers:Pin_Header_Straight_1x01_Pitch1.00mm" H 1100 15850 50  0001 C CNN
@@
 $Comp
 L STM32F413R(G-H)Tx_u U12
-U 2 1 5AFDDDDE
-P 13850 11850
-F 0 "U12" H 13850 11950 50  0000 C CNN
-F 1 "STM32F413R(G-H)Tx_u" H 13850 11750 50  0000 C CNN
-F 2 "Housings_QFP:LQFP-64_10x10mm_Pitch0.5mm" H 13850 11650 50  0000 C CIN
-F 3 "" H 13850 11850 50  0000 C CNN
-	2    13850 11850
+U 7 1 5AFDDDDE
+P 13050 8500
+F 0 "U12" H 13050 8600 50  0000 C CNN
+F 1 "STM32F413R(G-H)Tx_u" H 13050 8400 50  0000 C CNN
+F 2 "Housings_QFP:LQFP-64_10x10mm_Pitch0.5mm" H 13050 8300 50  0000 C CIN
+F 3 "" H 13050 8500 50  0000 C CNN
+	7    13050 8500
 	1    0    0    -1
 $EndComp
 $Comp
 L STM32F413R(G-H)Tx_u U12
-U 3 1 5AFDE42E
-P 13700 10000
-F 0 "U12" H 13700 10100 50  0000 C CNN
-F 1 "STM32F413R(G-H)Tx_u" H 13700 9900 50  0000 C CNN
-F 2 "Housings_QFP:LQFP-64_10x10mm_Pitch0.5mm" H 13700 9800 50  0000 C CIN
-F 3 "" H 13700 10000 50  0000 C CNN
-	3    13700 10000
+U 6 1 5AFDE42E
+P 14500 8550
+F 0 "U12" H 14500 8650 50  0000 C CNN
+F 1 "STM32F413R(G-H)Tx_u" H 14500 8450 50  0000 C CNN
+F 2 "Housings_QFP:LQFP-64_10x10mm_Pitch0.5mm" H 14500 8350 50  0000 C CIN
+F 3 "" H 14500 8550 50  0000 C CNN
+	6    14500 8550
 	1    0    0    -1
 $EndComp
 $Comp
 L STM32F413R(G-H)Tx_u U12
-U 4 1 5AFDE541
-P 16650 8050
-F 0 "U12" H 16650 8150 50  0000 C CNN
-F 1 "STM32F413R(G-H)Tx_u" H 16650 7950 50  0000 C CNN
-F 2 "Housings_QFP:LQFP-64_10x10mm_Pitch0.5mm" H 16650 7850 50  0000 C CIN
-F 3 "" H 16650 8050 50  0000 C CNN
-	4    16650 8050
+U 1 1 5AFDE541
+P 13750 13750
+F 0 "U12" H 13750 13850 50  0000 C CNN
+F 1 "STM32F413R(G-H)Tx_u" H 13750 13650 50  0000 C CNN
+F 2 "Housings_QFP:LQFP-64_10x10mm_Pitch0.5mm" H 13750 13550 50  0000 C CIN
+F 3 "" H 13750 13750 50  0000 C CNN
+	1    13750 13750
 	1    0    0    -1
 $EndComp
@@
 $Comp
 L STM32F413R(G-H)Tx_u U12
-U 1 1 5AFDE944
-P 13750 13750
-F 0 "U12" H 13750 13850 50  0000 C CNN
-F 1 "STM32F413R(G-H)Tx_u" H 13750 13650 50  0000 C CNN
-F 2 "Housings_QFP:LQFP-64_10x10mm_Pitch0.5mm" H 13750 13550 50  0000 C CIN
-F 3 "" H 13750 13750 50  0000 C CNN
-	1    13750 13750
-	1    0    0    -1
-$EndComp
-$Comp
-L STM32F413R(G-H)Tx_u U12
-U 6 1 5AFDEA93
-P 14500 8550
-F 0 "U12" H 14500 8650 50  0000 C CNN
-F 1 "STM32F413R(G-H)Tx_u" H 14500 8450 50  0000 C CNN
-F 2 "Housings_QFP:LQFP-64_10x10mm_Pitch0.5mm" H 14500 8350 50  0000 C CIN
-F 3 "" H 14500 8550 50  0000 C CNN
-	6    14500 8550
-	1    0    0    -1
-$EndComp
-$Comp
-L STM32F413R(G-H)Tx_u U12
-U 7 1 5AFDECD6
-P 13050 8500
-F 0 "U12" H 13050 8600 50  0000 C CNN
-F 1 "STM32F413R(G-H)Tx_u" H 13050 8400 50  0000 C CNN
-F 2 "Housings_QFP:LQFP-64_10x10mm_Pitch0.5mm" H 13050 8300 50  0000 C CIN
-F 3 "" H 13050 8500 50  0000 C CNN
-	7    13050 8500
-	1    0    0    -1
-$EndComp
-$Comp
-L STM32F413R(G-H)Tx_u U12
-U 8 1 5AFDEE64
+U 8 1 5AFDE944
 P 11450 8500
 F 0 "U12" H 11450 8600 50  0000 C CNN
@@
 F 3 "" H 11450 8500 50  0000 C CNN
 	8    11450 8500
+	1    0    0    -1
+$EndComp
+$Comp
+L STM32F413R(G-H)Tx_u U12
+U 4 1 5AFDEA93
+P 17100 8050
+F 0 "U12" H 17100 8150 50  0000 C CNN
+F 1 "STM32F413R(G-H)Tx_u" H 17100 7950 50  0000 C CNN
+F 2 "Housings_QFP:LQFP-64_10x10mm_Pitch0.5mm" H 17100 7850 50  0000 C CIN
+F 3 "" H 17100 8050 50  0000 C CNN
+	4    17100 8050
+	1    0    0    -1
+$EndComp
+$Comp
+L STM32F413R(G-H)Tx_u U12
+U 3 1 5AFDECD6
+P 13700 10000
+F 0 "U12" H 13700 10100 50  0000 C CNN
+F 1 "STM32F413R(G-H)Tx_u" H 13700 9900 50  0000 C CNN
+F 2 "Housings_QFP:LQFP-64_10x10mm_Pitch0.5mm" H 13700 9800 50  0000 C CIN
+F 3 "" H 13700 10000 50  0000 C CNN
+	3    13700 10000
+	1    0    0    -1
+$EndComp
+$Comp
+L STM32F413R(G-H)Tx_u U12
+U 2 1 5AFDEE64
+P 13850 11850
+F 0 "U12" H 13850 11950 50  0000 C CNN
+F 1 "STM32F413R(G-H)Tx_u" H 13850 11750 50  0000 C CNN
+F 2 "Housings_QFP:LQFP-64_10x10mm_Pitch0.5mm" H 13850 11650 50  0000 C CIN
+F 3 "" H 13850 11850 50  0000 C CNN
+	2    13850 11850
 	1    0    0    -1
 $EndComp
@@
 $EndComp
 Text Label 12200 2250 0    60   ~ 0
-SWIO
+SWDIO
 Text Label 12200 2350 0    60   ~ 0
 SWCLK
@@
 	1    0    0    -1
 $EndComp
+Text Label 15050 3600 0    60   ~ 0
+D+
 Text Label 15050 3400 0    60   ~ 0
-D+
-Text Label 15050 3600 0    60   ~ 0
 D-
 $Comp
@@
 	12000 8700 12000 8950
 Wire Wire Line
-	12000 8950 12200 8950
+	11900 8950 12200 8950
 Wire Wire Line
 	12500 8050 12600 8050
@@
 Wire Wire Line
 	13050 3500 13500 3500
-Wire Wire Line
-	13050 3400 13900 3400
 Wire Wire Line
 	12550 3200 12550 3000
@@
 $EndComp
 Wire Wire Line
-	13500 3500 13500 3600
-Wire Wire Line
-	13500 3600 13900 3600
-Wire Wire Line
 	14800 3400 15050 3400
 Wire Wire Line
 	14800 3600 15050 3600
+$Comp
+L TEST TP18
+U 1 1 5B06AA0D
+P 2400 15200
+F 0 "TP18" H 2400 15500 50  0000 C BNN
+F 1 "TEST" H 2400 15450 50  0000 C CNN
+F 2 "Pin_Headers:Pin_Header_Straight_1x01_Pitch1.00mm" H 2400 15200 50  0001 C CNN
+F 3 "" H 2400 15200 50  0001 C CNN
+	1    2400 15200
+	0    -1   -1   0
+$EndComp
+Text Label 2650 15200 0    61   ~ 0
+SYSCLK_OUT
+Wire Wire Line
+	2650 15200 2400 15200
+$Comp
+L +3.3V #PWR0100
+U 1 1 5B073ADE
+P 11950 8050
+F 0 "#PWR0100" H 11950 7900 50  0001 C CNN
+F 1 "+3.3V" H 11950 8190 50  0000 C CNN
+F 2 "" H 11950 8050 50  0001 C CNN
+F 3 "" H 11950 8050 50  0001 C CNN
+	1    11950 8050
+	1    0    0    -1
+$EndComp
+$Comp
+L +3.3V #PWR0101
+U 1 1 5B073CAB
+P 12050 8250
+F 0 "#PWR0101" H 12050 8100 50  0001 C CNN
+F 1 "+3.3V" H 12050 8390 50  0000 C CNN
+F 2 "" H 12050 8250 50  0001 C CNN
+F 3 "" H 12050 8250 50  0001 C CNN
+	1    12050 8250
+	1    0    0    -1
+$EndComp
+$Comp
+L +3.3V #PWR0102
+U 1 1 5B074042
+P 12050 8500
+F 0 "#PWR0102" H 12050 8350 50  0001 C CNN
+F 1 "+3.3V" H 12050 8640 50  0000 C CNN
+F 2 "" H 12050 8500 50  0001 C CNN
+F 3 "" H 12050 8500 50  0001 C CNN
+	1    12050 8500
+	1    0    0    -1
+$EndComp
+$Comp
+L +3.3V #PWR0103
+U 1 1 5B07420F
+P 12050 8750
+F 0 "#PWR0103" H 12050 8600 50  0001 C CNN
+F 1 "+3.3V" H 12050 8890 50  0000 C CNN
+F 2 "" H 12050 8750 50  0001 C CNN
+F 3 "" H 12050 8750 50  0001 C CNN
+	1    12050 8750
+	-1   0    0    1
+$EndComp
+$Comp
+L +3.3V #PWR0104
+U 1 1 5B0745A8
+P 11900 8950
+F 0 "#PWR0104" H 11900 8800 50  0001 C CNN
+F 1 "+3.3V" H 11900 9090 50  0000 C CNN
+F 2 "" H 11900 8950 50  0001 C CNN
+F 3 "" H 11900 8950 50  0001 C CNN
+	1    11900 8950
+	0    -1   -1   0
+$EndComp
+Connection ~ 12000 8950
+Wire Wire Line
+	13500 3500 13500 3400
+Wire Wire Line
+	13500 3400 13900 3400
+Wire Wire Line
+	13050 3400 13300 3400
+Wire Wire Line
+	13300 3400 13300 3600
+Wire Wire Line
+	13300 3600 13900 3600
+$Comp
+L C C50
+U 1 1 5B073098
+P 2000 2800
+F 0 "C50" H 2025 2900 50  0000 L CNN
+F 1 "100n" H 2025 2700 50  0000 L CNN
+F 2 "Capacitors_SMD:C_0603" H 2038 2650 50  0001 C CNN
+F 3 "" H 2000 2800 50  0001 C CNN
+	1    2000 2800
+	0    1    1    0
+$EndComp
+Wire Wire Line
+	2550 2800 2150 2800
+$Comp
+L GNDREF #PWR?
+U 1 1 5B0735C2
+P 1650 2800
+F 0 "#PWR?" H 1650 2550 50  0001 C CNN
+F 1 "GNDREF" H 1650 2650 50  0000 C CNN
+F 2 "" H 1650 2800 50  0001 C CNN
+F 3 "" H 1650 2800 50  0001 C CNN
+	1    1650 2800
+	0    1    1    0
+$EndComp
+Wire Wire Line
+	1650 2800 1850 2800
+$Comp
+L GNDREF #PWR?
+U 1 1 5B074522
+P 1800 3900
+F 0 "#PWR?" H 1800 3650 50  0001 C CNN
+F 1 "GNDREF" H 1800 3750 50  0000 C CNN
+F 2 "" H 1800 3900 50  0001 C CNN
+F 3 "" H 1800 3900 50  0001 C CNN
+	1    1800 3900
+	1    0    0    -1
+$EndComp
+$Comp
+L C C51
+U 1 1 5B074528
+P 2200 4450
+F 0 "C51" H 2225 4550 50  0000 L CNN
+F 1 "100n" H 2225 4350 50  0000 L CNN
+F 2 "Capacitors_SMD:C_0603" H 2238 4300 50  0001 C CNN
+F 3 "" H 2200 4450 50  0001 C CNN
+	1    2200 4450
+	0    1    1    0
+$EndComp
+Wire Wire Line
+	2750 4450 2350 4450
+$Comp
+L GNDREF #PWR?
+U 1 1 5B07452F
+P 1850 4450
+F 0 "#PWR?" H 1850 4200 50  0001 C CNN
+F 1 "GNDREF" H 1850 4300 50  0000 C CNN
+F 2 "" H 1850 4450 50  0001 C CNN
+F 3 "" H 1850 4450 50  0001 C CNN
+	1    1850 4450
+	0    1    1    0
+$EndComp
+Wire Wire Line
+	1850 4450 2050 4450
 $EndSCHEMATC
