File: Hardware/Elektrische_Komm.sch (KiCad schematic (older format))
At the start: 136 parts, among them J1 Conn_01x01, J2 Conn_01x01, J3 Conn_01x01, J4 Conn_01x04, J5 USB_OTG, Q1 BSZ014NE2LS5IF, Q10 BSR202NL6327HTSA1, Q11 BSR202NL6327HTSA1, Q12 BSR202NL6327HTSA1, Q13 BSR202NL6327HTSA1, Q14 BSR202NL6327HTSA1, Q2 BSZ014NE2LS5IF, Q3 BSZ014NE2LS5IF, Q4 BSZ014NE2LS5IF, Q5 BSZ014NE2LS5IF, Q6 BSZ014NE2LS5IF, Q7 BSR202NL6327HTSA1, Q8 BSR202NL6327HTSA1, Q9 BSR202NL6327HTSA1, SW1 SW_Push, SW2 SW_Push, U1 TS374IDT, U10 TPS561201, U11 LVM339IDT, U12 STM32F413R(G-H)Tx_u, U2 UCC27710, U3 ACS723LLCTR, U4 UCC27710, U5 ACS723LLCTR, U6 UCC27710, U7 74HC32D, U8 74LVC2G02, U9 LDK715M50R, Y1 10MHz

Commit message: _______________ < Neue Bauteile >  ---------------       \                    / \  //\        \    |\___/|      /   \//  \\             /0  0  \__  /    //  | \ \            /     /  \/_/    //   |  \  \            @_^_@'/   \/_   //    |   \   \            //_^_/     \/_ //     |    \    \         ( //) |        \///      |     \     \       ( / /) _|_ /   )  //       |      \     _\     ( // /) '/,_ _ _/  ( ; -.    |    _ _\.-~        .-~~~^-.   (( / / )) ,-{        _      `-.|.-~-.           .~         `.  (( // / ))  '/\      /                 ~-. _ .-~      .-~^-.  \  (( /// ))      `.   {            }                   /      \  \   (( / ))     .----~-.\        \-'                 .~         \  `. \^-.              ///.----..>        \             _ -~             `.  ^-`  ^-_                ///-._ _ _ _ _ _ _}^ - - - - ~                     ~-- ,.-~                                                                   /.-~
Parts:
- removed C14, C51: 100n, Capacitors_SMD:C_0603, symbol C
- removed C15: 470n, Capacitors_SMD:C_0603, symbol C
- removed C9: 10n, Capacitors_SMD:C_0603, symbol C
- removed R11, R15, R20, R21, R33, R34: R, Resistors_SMD:R_0603, symbol R
- removed R12, R14: 27, Resistors_SMD:R_0603, symbol R
- removed R32, R40: 10k, Resistors_SMD:R_0603, symbol R
- removed R8: 1,5k, Resistors_SMD:R_0603, symbol R
- removed U11: LVM339IDT, Housings_SOIC:SOIC-14_3.9x8.7mm_Pitch1.27mm, symbol LVM339IDT
- removed U5: ACS723LLCTR, Housings_SOIC:SOIC-8_3.9x4.9mm_Pitch1.27mm, symbol ACS723LLCTR
- removed unit 2 of U7
- removed U9: LDK715M50R, TO_SOT_Packages_SMD:SOT-23-5_HandSoldering, symbol LDK715M50R
- added R50, R51: R, Resistors_SMD:R_0603, symbol R
- added TP22, TP23, TP24, TP25: TEST, Pin_Headers:Pin_Header_Straight_1x01_Pitch1.00mm, symbol TEST
- added U11: TLC352, Housings_SSOP:TSSOP-8_4.4x3mm_Pitch0.65mm, symbol TLC352
- Y1: value 10MHz -> 24MHz
Connections:
- net labels added: Meas_out, StopMCU, ZK_Out
- net labels removed: +5V, Curr_direct_B, Curr_mcu_A, OR2
- wire segments 438 -> 378
Other:
- moved on the sheet: TP1

Commit message: _______________________ < Layout weitergeführt >  -----------------------       \                    / \  //\        \    |\___/|      /   \//  \\             /0  0  \__  /    //  | \ \            /     /  \/_/    //   |  \  \            @_^_@'/   \/_   //    |   \   \            //_^_/     \/_ //     |    \    \         ( //) |        \///      |     \     \       ( / /) _|_ /   )  //       |      \     _\     ( // /) '/,_ _ _/  ( ; -.    |    _ _\.-~        .-~~~^-.   (( / / )) ,-{        _      `-.|.-~-.           .~         `.  (( // / ))  '/\      /                 ~-. _ .-~      .-~^-.  \  (( /// ))      `.   {            }                   /      \  \   (( / ))     .----~-.\        \-'                 .~         \  `. \^-.              ///.----..>        \             _ -~             `.  ^-`  ^-_                ///-._ _ _ _ _ _ _}^ - - - - ~                     ~-- ,.-~                                                                   /.-~
Parts:
- D1, D3, D5: footprint kicadBibs:SOD-123W -> Diodes_SMD:D_SOD-123F
Connections:
- net A: now also C2.2, U1.4 (-), U2.6 (HS)
- net A_conn: no longer C2.2, U1.4 (-), U2.6 (HS)
- net B: now also C5.2, U1.6 (-), U4.6 (HS)
- net B_conn: no longer C5.2, U1.6 (-), U4.6 (HS)
- net Bemf_A: now also U12.43 (PA10/DFSDM2_DATIN3/I2S2_SD/I2S5_SD/SPI2_MOSI/SPI5_MOSI/TIM1_CH3/USART1_RX/USB_OTG_FS_ID); no longer U12.41 (PA8/CAN3_RX/DFSDM1_CKOUT/I2C3_SCL/RCC_MCO_1/SDIO_D1/TIM1_CH1/UART7_RX/USART1_CK/USB_OTG_FS_SOF)
- net Bemf_C: now also U12.41 (PA8/CAN3_RX/DFSDM1_CKOUT/I2C3_SCL/RCC_MCO_1/SDIO_D1/TIM1_CH1/UART7_RX/USART1_CK/USB_OTG_FS_SOF); no longer U12.43 (PA10/DFSDM2_DATIN3/I2S2_SD/I2S5_SD/SPI2_MOSI/SPI5_MOSI/TIM1_CH3/USART1_RX/USB_OTG_FS_ID)
- net DCDC_EN renamed VCC
Other:
- note added: "Strommessung\n"

Commit message: _______________________________ < K_ind Berechnung hinzugefügt >  -------------------------------       \                    / \  //\        \    |\___/|      /   \//  \\             /0  0  \__  /    //  | \ \            /     /  \/_/    //   |  \  \            @_^_@'/   \/_   //    |   \   \            //_^_/     \/_ //     |    \    \         ( //) |        \///      |     \     \       ( / /) _|_ /   )  //       |      \     _\     ( // /) '/,_ _ _/  ( ; -.    |    _ _\.-~        .-~~~^-.   (( / / )) ,-{        _      `-.|.-~-.           .~         `.  (( // / ))  '/\      /                 ~-. _ .-~      .-~^-.  \  (( /// ))      `.   {            }                   /      \  \   (( / ))     .----~-.\        \-'                 .~         \  `. \^-.              ///.----..>        \             _ -~             `.  ^-`  ^-_                ///-._ _ _ _ _ _ _}^ - - - - ~                     ~-- ,.-~                                                                   /.-~
Connections:
- net Curr_mcu_B: no longer names the net of U12.25 (PC5/ADC1_IN15/DFSDM2_DATIN2/FMPI2C1_SMBA/FSMC_NOE/QUADSPI_BK2_IO3/USART3_RX)
Changed lines of the file:
@@
 Text Label 17050 13550 0    61   ~ 0
 HI_A
-Text Label 16900 9700 0    60   ~ 0
-Curr_mcu_B
 Text Label 17050 13350 0    61   ~ 0
 DAC1
@@
 	16600 9400 16900 9400
 Wire Wire Line
-	16900 9700 16600 9700
-Wire Wire Line
 	16900 9600 16600 9600

Commit message: ______________________ < Layout weitergemacht >  ----------------------       \                    / \  //\        \    |\___/|      /   \//  \\             /0  0  \__  /    //  | \ \            /     /  \/_/    //   |  \  \            @_^_@'/   \/_   //    |   \   \            //_^_/     \/_ //     |    \    \         ( //) |        \///      |     \     \       ( / /) _|_ /   )  //       |      \     _\     ( // /) '/,_ _ _/  ( ; -.    |    _ _\.-~        .-~~~^-.   (( / / )) ,-{        _      `-.|.-~-.           .~         `.  (( // / ))  '/\      /                 ~-. _ .-~      .-~^-.  \  (( /// ))      `.   {            }                   /      \  \   (( / ))     .----~-.\        \-'                 .~         \  `. \^-.              ///.----..>        \             _ -~             `.  ^-`  ^-_                ///-._ _ _ _ _ _ _}^ - - - - ~                     ~-- ,.-~                                                                   /.-~
Parts:
- R18, R5, R9: footprint Resistors_SMD:R_0603 -> Resistors_SMD:R_1210
Connections:
- net +15V is gone; now on net VCC: R18.2, R5.2, R9.2
- net A_conn is gone; now on net A: TP2.1
- net B_conn is gone; now on net B: TP3.1
- net A: no longer U12.8 (PC0/ADC1_IN10/DFSDM2_CKIN4/LPTIM1_IN1/SAI1_MCLK_B/SYS_WKUP2)
- net B: no longer U12.9 (PC1/ADC1_IN11/DFSDM2_DATIN4/LPTIM1_OUT/SAI1_SD_B/SYS_WKUP3)
- net C: no longer U12.10 (PC2/ADC1_IN12/DFSDM1_CKOUT/DFSDM2_DATIN7/FSMC_NWE/I2S2_ext_SD/LPTIM1_IN2/SAI1_SCK_B/SPI2_MISO)
- net Sternpunkt_virtuell: no longer U12.11 (PC3/ADC1_IN13/DFSDM2_CKIN7/FSMC_A0/I2S2_SD/LPTIM1_ETR/SAI1_FS_B/SPI2_MOSI)
- no-connect marks 0 -> 1
Other:
- moved on the sheet: R41, R42, SW1, SW2
Changed lines of the file:
@@
 F 0 "R5" V 6880 1700 50  0000 C CNN
 F 1 "3" V 6800 1700 50  0000 C CNN
-F 2 "Resistors_SMD:R_0603" V 6730 1700 50  0001 C CNN
+F 2 "Resistors_SMD:R_1210" V 6730 1700 50  0001 C CNN
 F 3 "" H 6800 1700 50  0001 C CNN
 	1    6800 1700
@@
 HO_A
 $Comp
-L +15V #PWR08
-U 1 1 5AF34250
-P 6550 1700
-F 0 "#PWR08" H 6550 1550 50  0001 C CNN
-F 1 "+15V" H 6550 1840 50  0000 C CNN
-F 2 "" H 6550 1700 50  0001 C CNN
-F 3 "" H 6550 1700 50  0001 C CNN
-	1    6550 1700
-	0    -1   -1   0
-$EndComp
-$Comp
 L UCC27710 U4
 U 1 1 5AF34890
@@
 F 0 "R9" V 6930 3150 50  0000 C CNN
 F 1 "3" V 6850 3150 50  0000 C CNN
-F 2 "Resistors_SMD:R_0603" V 6780 3150 50  0001 C CNN
+F 2 "Resistors_SMD:R_1210" V 6780 3150 50  0001 C CNN
 F 3 "" H 6850 3150 50  0001 C CNN
 	1    6850 3150
@@
 LO_B
 $Comp
-L +15V #PWR011
-U 1 1 5AF348CB
-P 6600 3150
-F 0 "#PWR011" H 6600 3000 50  0001 C CNN
-F 1 "+15V" H 6600 3290 50  0000 C CNN
-F 2 "" H 6600 3150 50  0001 C CNN
-F 3 "" H 6600 3150 50  0001 C CNN
-	1    6600 3150
-	0    -1   -1   0
-$EndComp
-$Comp
 L UCC27710 U6
 U 1 1 5AF3595A
@@
 F 0 "R18" V 6930 4550 50  0000 C CNN
 F 1 "3" V 6850 4550 50  0000 C CNN
-F 2 "Resistors_SMD:R_0603" V 6780 4550 50  0001 C CNN
+F 2 "Resistors_SMD:R_1210" V 6780 4550 50  0001 C CNN
 F 3 "" H 6850 4550 50  0001 C CNN
 	1    6850 4550
@@
 Text Label 7550 5150 0    60   ~ 0
 LO_C
-$Comp
-L +15V #PWR014
-U 1 1 5AF35995
-P 6600 4550
-F 0 "#PWR014" H 6600 4400 50  0001 C CNN
-F 1 "+15V" H 6600 4690 50  0000 C CNN
-F 2 "" H 6600 4550 50  0001 C CNN
-F 3 "" H 6600 4550 50  0001 C CNN
-	1    6600 4550
-	0    -1   -1   0
-$EndComp
 Text Label 2400 1100 0    60   ~ 0
 HO_B
@@
 $EndComp
 Text Label 1350 13300 0    60   ~ 0
-A_conn
+A
 Text Label 1350 13500 0    60   ~ 0
-B_conn
+B
 Text Label 1350 13700 0    60   ~ 0
 C
@@
 L R R41
 U 1 1 5B0082F6
-P 7550 14750
-F 0 "R41" V 7630 14750 50  0000 C CNN
-F 1 "1k" V 7550 14750 50  0000 C CNN
-F 2 "Resistors_SMD:R_0603" V 7480 14750 50  0001 C CNN
-F 3 "" H 7550 14750 50  0001 C CNN
-	1    7550 14750
-	0    -1   -1   0
+P 4750 14150
+F 0 "R41" V 4830 14150 50  0000 C CNN
+F 1 "1k" V 4750 14150 50  0000 C CNN
+F 2 "Resistors_SMD:R_0603" V 4680 14150 50  0001 C CNN
+F 3 "" H 4750 14150 50  0001 C CNN
+	1    4750 14150
+	1    0    0    -1
 $EndComp
 $Comp
 L +3.3V #PWR062
 U 1 1 5B00880E
-P 7250 14750
-F 0 "#PWR062" H 7250 14600 50  0001 C CNN
-F 1 "+3.3V" H 7250 14890 50  0000 C CNN
-F 2 "" H 7250 14750 50  0001 C CNN
-F 3 "" H 7250 14750 50  0001 C CNN
-	1    7250 14750
-	0    -1   -1   0
+P 4750 13850
+F 0 "#PWR062" H 4750 13700 50  0001 C CNN
+F 1 "+3.3V" H 4750 13990 50  0000 C CNN
+F 2 "" H 4750 13850 50  0001 C CNN
+F 3 "" H 4750 13850 50  0001 C CNN
+	1    4750 13850
+	1    0    0    -1
 $EndComp
 $Comp
 L SW_Push SW1
 U 1 1 5B008F37
-P 8050 14750
-F 0 "SW1" H 8100 14850 50  0000 L CNN
-F 1 "SW_Push" H 8050 14690 50  0000 C CNN
-F 2 "kicadBibs:Switch" H 8050 14950 50  0001 C CNN
-F 3 "" H 8050 14950 50  0001 C CNN
-	1    8050 14750
-	1    0    0    -1
+P 4750 14650
+F 0 "SW1" H 4800 14750 50  0000 L CNN
+F 1 "SW_Push" H 4750 14590 50  0000 C CNN
+F 2 "kicadBibs:Switch" H 4750 14850 50  0001 C CNN
+F 3 "" H 4750 14850 50  0001 C CNN
+	1    4750 14650
+	0    1    1    0
 $EndComp
 $Comp
 L GNDREF #PWR063
 U 1 1 5B009068
-P 8450 14750
-F 0 "#PWR063" H 8450 14500 50  0001 C CNN
-F 1 "GNDREF" H 8450 14600 50  0000 C CNN
-F 2 "" H 8450 14750 50  0001 C CNN
-F 3 "" H 8450 14750 50  0001 C CNN
-	1    8450 14750
-	0    -1   -1   0
+P 4750 15050
+F 0 "#PWR063" H 4750 14800 50  0001 C CNN
+F 1 "GNDREF" H 4750 14900 50  0000 C CNN
+F 2 "" H 4750 15050 50  0001 C CNN
+F 3 "" H 4750 15050 50  0001 C CNN
+	1    4750 15050
+	1    0    0    -1
 $EndComp
-Text Label 7750 14500 1    61   ~ 0
+Text Label 5000 14350 0    61   ~ 0
 NRST
-Text Label 16900 9200 0    60   ~ 0
-A
-Text Label 16900 9300 0    60   ~ 0
-B
-Text Label 16900 9400 0    60   ~ 0
-C
 $Comp
 L R R42
 U 1 1 5AFE0658
-P 10100 14750
-F 0 "R42" V 10180 14750 50  0000 C CNN
-F 1 "1k" V 10100 14750 50  0000 C CNN
-F 2 "Resistors_SMD:R_0603" V 10030 14750 50  0001 C CNN
-F 3 "" H 10100 14750 50  0001 C CNN
-	1    10100 14750
-	0    -1   -1   0
+P 5850 14700
+F 0 "R42" V 5930 14700 50  0000 C CNN
+F 1 "1k" V 5850 14700 50  0000 C CNN
+F 2 "Resistors_SMD:R_0603" V 5780 14700 50  0001 C CNN
+F 3 "" H 5850 14700 50  0001 C CNN
+	1    5850 14700
+	1    0    0    -1
 $EndComp
 $Comp
 L +3.3V #PWR064
 U 1 1 5AFE065E
-P 9250 14750
-F 0 "#PWR064" H 9250 14600 50  0001 C CNN
-F 1 "+3.3V" H 9250 14890 50  0000 C CNN
-F 2 "" H 9250 14750 50  0001 C CNN
-F 3 "" H 9250 14750 50  0001 C CNN
-	1    9250 14750
-	0    -1   -1   0
+P 5850 13700
+F 0 "#PWR064" H 5850 13550 50  0001 C CNN
+F 1 "+3.3V" H 5850 13840 50  0000 C CNN
+F 2 "" H 5850 13700 50  0001 C CNN
+F 3 "" H 5850 13700 50  0001 C CNN
+	1    5850 13700
+	1    0    0    -1
 $EndComp
 $Comp
 L SW_Push SW2
 U 1 1 5AFE0665
-P 9600 14750
-F 0 "SW2" H 9650 14850 50  0000 L CNN
-F 1 "SW_Push" H 9600 14690 50  0000 C CNN
-F 2 "kicadBibs:Switch" H 9600 14950 50  0001 C CNN
-F 3 "" H 9600 14950 50  0001 C CNN
-	1    9600 14750
-	1    0    0    -1
+P 5850 14050
+F 0 "SW2" H 5900 14150 50  0000 L CNN
+F 1 "SW_Push" H 5850 13990 50  0000 C CNN
+F 2 "kicadBibs:Switch" H 5850 14250 50  0001 C CNN
+F 3 "" H 5850 14250 50  0001 C CNN
+	1    5850 14050
+	0    1    1    0
 $EndComp
 $Comp
 L GNDREF #PWR065
 U 1 1 5AFE066B
-P 10550 14750
-F 0 "#PWR065" H 10550 14500 50  0001 C CNN
-F 1 "GNDREF" H 10550 14600 50  0000 C CNN
-F 2 "" H 10550 14750 50  0001 C CNN
-F 3 "" H 10550 14750 50  0001 C CNN
-	1    10550 14750
-	0    -1   -1   0
+P 5850 15050
+F 0 "#PWR065" H 5850 14800 50  0001 C CNN
+F 1 "GNDREF" H 5850 14900 50  0000 C CNN
+F 2 "" H 5850 15050 50  0001 C CNN
+F 3 "" H 5850 15050 50  0001 C CNN
+	1    5850 15050
+	1    0    0    -1
 $EndComp
-Text Label 9850 14500 1    61   ~ 0
+Text Label 6600 14400 2    61   ~ 0
 Freigabe_button
 Text Label 17100 11650 0    60   ~ 0
 Freigabe_MCU
-Text Label 16900 9500 0    60   ~ 0
-Sternpunkt_virtuell
 Text Notes 2550 15850 0    98   ~ 0
 Testpunkte
@@
 	5600 1650 5600 1850
 Wire Wire Line
-	6550 1700 6650 1700
+	6500 1700 6650 1700
 Wire Wire Line
 	6050 3900 6050 3750
@@
 	5650 3300 5650 3250
 Wire Wire Line
-	6600 3150 6700 3150
+	6450 3150 6700 3150
 Wire Wire Line
 	6050 5300 6050 5150
@@
 	5650 4700 5650 4650
 Wire Wire Line
-	6600 4550 6700 4550
+	6450 4550 6700 4550
 Wire Wire Line
 	2400 1100 2700 1100
@@
 	17050 13950 16750 13950
 Wire Wire Line
-	16600 9200 16900 9200
-Wire Wire Line
-	16900 9300 16600 9300
-Wire Wire Line
 	17050 13350 16750 13350
 Wire Wire Line
@@
 Connection ~ 18350 8500
 Wire Wire Line
-	7250 14750 7400 14750
+	4750 13850 4750 14000
 Wire Wire Line
-	8450 14750 8250 14750
+	4750 15050 4750 14850
 Wire Wire Line
-	7700 14750 7850 14750
+	4750 14300 4750 14450
 Wire Wire Line
-	7750 14500 7750 14750
-Connection ~ 7750 14750
-Wire Wire Line
-	16600 9400 16900 9400
+	5000 14350 4750 14350
+Connection ~ 4750 14350
 Wire Wire Line
 	16900 9600 16600 9600
 Wire Wire Line
-	9250 14750 9400 14750
-Wire Wire Line
-	10250 14750 10550 14750
-Wire Wire Line
-	9800 14750 9950 14750
-Wire Wire Line
-	9850 14500 9850 14750
-Connection ~ 9850 14750
-Wire Wire Line
 	17100 11650 16950 11650
 Wire Wire Line
-	16900 9500 16600 9500
-Wire Wire Line
 	2400 14300 2650 14300
 Wire Wire Line
@@
 Text Label 13450 6700 0    60   ~ 0
 VCC
+NoConn ~ 5850 14000
+Wire Wire Line
+	5850 13850 5850 13700
+Wire Wire Line
+	5850 15050 5850 14850
+Wire Wire Line
+	5850 14550 5850 14250
+Wire Wire Line
+	6600 14400 5850 14400
+Connection ~ 5850 14400
+Wire Notes Line
+	6700 13050 6700 16100
+Text Label 6500 1700 0    60   ~ 0
+VCC
+Text Label 6450 3150 0    60   ~ 0
+VCC
+Text Label 6450 4550 0    60   ~ 0
+VCC
 $EndSCHEMATC

Commit message: ___________________ < MOSFETS geändert >  -------------------       \                    / \  //\        \    |\___/|      /   \//  \\             /0  0  \__  /    //  | \ \            /     /  \/_/    //   |  \  \            @_^_@'/   \/_   //    |   \   \            //_^_/     \/_ //     |    \    \         ( //) |        \///      |     \     \       ( / /) _|_ /   )  //       |      \     _\     ( // /) '/,_ _ _/  ( ; -.    |    _ _\.-~        .-~~~^-.   (( / / )) ,-{        _      `-.|.-~-.           .~         `.  (( // / ))  '/\      /                 ~-. _ .-~      .-~^-.  \  (( /// ))      `.   {            }                   /      \  \   (( / ))     .----~-.\        \-'                 .~         \  `. \^-.              ///.----..>        \             _ -~             `.  ^-`  ^-_                ///-._ _ _ _ _ _ _}^ - - - - ~                     ~-- ,.-~                                                                   /.-~
Parts:
- removed R28: 10k, Resistors_SMD:R_0603, symbol R
- removed R50, R51: R, Resistors_SMD:R_0603, symbol R
- removed U11: TLC352, Housings_SSOP:TSSOP-8_4.4x3mm_Pitch0.65mm, symbol TLC352
- removed U7: 74HC32D, Housings_SSOP:TSSOP-14_4.4x5mm_Pitch0.65mm, symbol 74HC32D
- added U5: MCP6546, TO_SOT_Packages_SMD:SOT-23-5, symbol MCP6561
- added U7: NC7WZ32, Housings_SSOP:VSSOP-8_2.3x2mm_Pitch0.5mm, symbol NC7WZ32
- Q1, Q2, Q3, Q4, Q5, Q6: value BSZ014NE2LS5IF -> CSD16556Q5B; footprint kicadBibs:SON65P330X330X110-8N -> kicadBibs:SON5x6
Connections:
- net +3V3: now also U5.5 (V+), U7.8 (V+)
- net Curr_direct_A: now also U5.3 (+)
- net Freigabe_MCU: now also U7.6
- net Freigabe_button: now also U7.5
- net GNDREF: now also U5.2 (V-), U7.4 (GND)
- net Stop: now also U7.7
- net StopMCU: now also U7.2
- net at R27.2: now also U7.3
- net Stop_Hardware: now reaches R22.2
- net Stop_Hardware: now also U5.1, U7.1
- net at R23.2, R25.1: now also U5.4 (-)
Other:
- moved on the sheet: C11

Commit message: _____________________ < BW_SEL hinzugefügt >  ---------------------       \                    / \  //\        \    |\___/|      /   \//  \\             /0  0  \__  /    //  | \ \            /     /  \/_/    //   |  \  \            @_^_@'/   \/_   //    |   \   \            //_^_/     \/_ //     |    \    \         ( //) |        \///      |     \     \       ( / /) _|_ /   )  //       |      \     _\     ( // /) '/,_ _ _/  ( ; -.    |    _ _\.-~        .-~~~^-.   (( / / )) ,-{        _      `-.|.-~-.           .~         `.  (( // / ))  '/\      /                 ~-. _ .-~      .-~^-.  \  (( /// ))      `.   {            }                   /      \  \   (( / ))     .----~-.\        \-'                 .~         \  `. \^-.              ///.----..>        \             _ -~             `.  ^-`  ^-_                ///-._ _ _ _ _ _ _}^ - - - - ~                     ~-- ,.-~                                                                   /.-~
Connections:
- net A: no longer TP2.1
- net B: no longer TP3.1
- net Bemf_A: now also TP2.1
- net Bemf_B: now also TP3.1
- net Bemf_C: now also TP5.1
- net C: no longer TP5.1
- net GNDREF: no longer U3.6 (BW_SEL)
- net BW_SEL: now reaches U12.17 (PA3/ADC1_IN3/FSMC_D5/FSMC_DA5/I2S2_MCK/SAI1_SD_B/TIM2_CH4/TIM5_CH4/TIM9_CH2/USART2_RX)
- net BW_SEL: now also U3.6 (BW_SEL)
Other:
- moved on the sheet: D4
Changed lines of the file:
@@
 	0    -1   -1   0
 $EndComp
-Text Label 1350 13300 0    60   ~ 0
-A
-Text Label 1350 13500 0    60   ~ 0
-B
-Text Label 1350 13700 0    60   ~ 0
-C
 Text Label 1350 13900 0    60   ~ 0
 HO_A
@@
 	1    0    0    -1
 $EndComp
-Text Label 15050 3400 0    60   ~ 0
+Text Label 13800 3300 0    60   ~ 0
 D+
-Text Label 15050 3600 0    60   ~ 0
+Text Label 13800 3500 0    60   ~ 0
 D-
 $Comp
 L USBLC6-2SC6Y D4
 U 1 1 5B005011
-P 14300 3700
-F 0 "D4" H 14300 3700 60  0000 C CNN
-F 1 "USBLC6-2SC6Y" H 14250 3600 60  0000 C CNN
-F 2 "TO_SOT_Packages_SMD:SOT-23-6" H 14300 3700 60  0001 C CNN
-F 3 "" H 14300 3700 60  0001 C CNN
-	1    14300 3700
+P 13050 3600
+F 0 "D4" H 13050 3600 60  0000 C CNN
+F 1 "USBLC6-2SC6Y" H 13000 3500 60  0000 C CNN
+F 2 "TO_SOT_Packages_SMD:SOT-23-6" H 13050 3600 60  0001 C CNN
+F 3 "" H 13050 3600 60  0001 C CNN
+	1    13050 3600
 	-1   0    0    -1
 $EndComp
@@
 L GNDREF #PWR060
 U 1 1 5B005DAE
-P 14800 3500
-F 0 "#PWR060" H 14800 3250 50  0001 C CNN
-F 1 "GNDREF" H 14800 3350 50  0001 C CNN
-F 2 "" H 14800 3500 50  0001 C CNN
-F 3 "" H 14800 3500 50  0001 C CNN
-	1    14800 3500
+P 13550 3400
+F 0 "#PWR060" H 13550 3150 50  0001 C CNN
+F 1 "GNDREF" H 13550 3250 50  0001 C CNN
+F 2 "" H 13550 3400 50  0001 C CNN
+F 3 "" H 13550 3400 50  0001 C CNN
+	1    13550 3400
 	0    -1   -1   0
 $EndComp
@@
 	2550 3000 2550 2800
 Wire Wire Line
-	2450 3200 2450 3550
+	2450 3300 2450 3550
 Wire Wire Line
 	2450 3300 2350 3300
@@
 	3000 3150 3000 3100
 Connection ~ 3000 3100
-Wire Wire Line
-	2350 3200 2450 3200
 Connection ~ 2450 3300
 Wire Notes Line
@@
 	1100 13900 1350 13900
 Wire Wire Line
-	1100 13700 1350 13700
-Wire Wire Line
-	1100 13500 1350 13500
-Wire Wire Line
-	1100 13300 1350 13300
+	1100 13700 1550 13700
+Wire Wire Line
+	1100 13500 1550 13500
+Wire Wire Line
+	1100 13300 1550 13300
 Wire Wire Line
 	2400 15550 2700 15550
@@
 Connection ~ 12050 4300
 Wire Wire Line
-	12350 3400 13900 3400
-Wire Wire Line
-	12350 3500 13500 3500
-Wire Wire Line
-	13700 3500 13900 3500
-Wire Wire Line
-	14800 3400 15050 3400
-Wire Wire Line
-	14800 3600 15050 3600
+	12450 3400 12650 3400
+Wire Wire Line
+	13550 3300 13800 3300
+Wire Wire Line
+	13550 3500 13800 3500
 Wire Wire Line
 	2650 15200 2400 15200
@@
 Curr_direct_A
 Wire Wire Line
-	12350 3200 13700 3200
-Wire Wire Line
-	13700 3200 13700 3500
-Wire Wire Line
-	13900 3600 13500 3600
-Wire Wire Line
-	13500 3600 13500 3500
-Wire Wire Line
 	17500 12050 16950 12050
 Wire Wire Line
@@
 	5850 15050 5850 14850
 Wire Wire Line
-	5850 14550 5850 14250
+	5850 14250 5850 14550
 Wire Wire Line
 	6600 14400 5850 14400
@@
 	5800 6000 5800 6100
 Connection ~ 6900 6100
+Text Label 1550 13300 0    60   ~ 0
+Bemf_A
+Text Label 1550 13500 0    60   ~ 0
+Bemf_B
+Text Label 1550 13700 0    60   ~ 0
+Bemf_C
+Wire Wire Line
+	12350 3300 12350 3400
+Wire Wire Line
+	12450 3400 12450 3200
+Wire Wire Line
+	12450 3200 12350 3200
+Wire Wire Line
+	12350 3300 12650 3300
+Wire Wire Line
+	12650 3500 12350 3500
+Text Label 2450 3200 0    60   ~ 0
+BW_SEL
+Wire Wire Line
+	2450 3200 2350 3200
+Text Label 17050 13250 0    60   ~ 0
+BW_SEL
+Wire Wire Line
+	16750 13250 17050 13250
 $EndSCHEMATC

Commit message: _________________ < Planes erledigt >  -----------------       \                    / \  //\        \    |\___/|      /   \//  \\             /0  0  \__  /    //  | \ \            /     /  \/_/    //   |  \  \            @_^_@'/   \/_   //    |   \   \            //_^_/     \/_ //     |    \    \         ( //) |        \///      |     \     \       ( / /) _|_ /   )  //       |      \     _\     ( // /) '/,_ _ _/  ( ; -.    |    _ _\.-~        .-~~~^-.   (( / / )) ,-{        _      `-.|.-~-.           .~         `.  (( // / ))  '/\      /                 ~-. _ .-~      .-~^-.  \  (( /// ))      `.   {            }                   /      \  \   (( / ))     .----~-.\        \-'                 .~         \  `. \^-.              ///.----..>        \             _ -~             `.  ^-`  ^-_                ///-._ _ _ _ _ _ _}^ - - - - ~                     ~-- ,.-~                                                                   /.-~
Parts:
- added C9: C, Capacitors_THT:CP_Radial_D10.0mm_P5.00mm, symbol C
- added J6, J7: Conn_01x01, kicadBibs:Laborbuchse, symbol Conn_01x01
- C6: footprint (none) -> Capacitors_THT:CP_Radial_D10.0mm_P5.00mm
- L1: footprint kicadBibs:NLCV32T-3R3M-EF -> kicadBibs:SRN3015-3R3M
Connections:
- net GNDREF: now also C9.2, J7.1 (Pin_1)
- net VCC: now also C9.1; no longer C6.1
- net Vin: now also J6.1 (Pin_1)
Other:
- moved on the sheet: C6, R16
