File: Hardware/Elektrische_Komm.sch (KiCad schematic (older format))
At the start: 125 parts, among them J1 Conn_01x01, J2 Conn_01x01, J3 Conn_01x01, J4 Conn_01x04, J5 USB_OTG, J6 Conn_01x01, J7 Conn_01x01, Q1 CSD16556Q5B, Q10 BSR202NL6327HTSA1, Q11 BSR202NL6327HTSA1, Q12 BSR202NL6327HTSA1, Q13 BSR202NL6327HTSA1, Q14 BSR202NL6327HTSA1, Q2 CSD16556Q5B, Q3 CSD16556Q5B, Q4 CSD16556Q5B, Q5 CSD16556Q5B, Q6 CSD16556Q5B, Q7 BSR202NL6327HTSA1, Q8 BSR202NL6327HTSA1, Q9 BSR202NL6327HTSA1, SW1 SW_Push, SW2 SW_Push, U1 TS374IDT, U10 TPS561201, U12 STM32F413R(G-H)Tx_u, U2 UCC27710, U3 ACS723LLCTR, U4 UCC27710, U5 MCP6546, U6 UCC27710, U7 NC7WZ32, U8 74LVC2G02, Y1 24MHz

Commit message: _____________________ < Layout Groundplanes >  ---------------------       \                    / \  //\        \    |\___/|      /   \//  \\             /0  0  \__  /    //  | \ \            /     /  \/_/    //   |  \  \            @_^_@'/   \/_   //    |   \   \            //_^_/     \/_ //     |    \    \         ( //) |        \///      |     \     \       ( / /) _|_ /   )  //       |      \     _\     ( // /) '/,_ _ _/  ( ; -.    |    _ _\.-~        .-~~~^-.   (( / / )) ,-{        _      `-.|.-~-.           .~         `.  (( // / ))  '/\      /                 ~-. _ .-~      .-~^-.  \  (( /// ))      `.   {            }                   /      \  \   (( / ))     .----~-.\        \-'                 .~         \  `. \^-.              ///.----..>        \             _ -~             `.  ^-`  ^-_                ///-._ _ _ _ _ _ _}^ - - - - ~                     ~-- ,.-~                                                                   /.-~
Parts:
- removed C9: C, Capacitors_THT:CP_Radial_D10.0mm_P5.00mm, symbol C
- removed D2: D, symbol D
Connections:
- net Vin is gone; now on net VCC: C1.1, J6.1 (Pin_1)
Changed lines of the file:
@@
 Text Label 4500 2750 0    60   ~ 0
 Vin
-$Comp
-L D D2
-U 1 1 5AF3A4A4
-P 4900 2750
-F 0 "D2" H 4900 2850 50  0000 C CNN
-F 1 "D" H 4900 2650 50  0000 C CNN
-F 2 "" H 4900 2750 50  0001 C CNN
-F 3 "" H 4900 2750 50  0001 C CNN
-	1    4900 2750
-	-1   0    0    1
-$EndComp
 Text Label 5150 2750 0    60   ~ 0
 VCC
@@
 Connection ~ 4650 3600
 Wire Wire Line
-	5150 2750 5050 2750
-Wire Wire Line
-	4500 2750 4750 2750
+	4500 2750 5150 2750
 Wire Wire Line
 	8650 1150 9600 1150
@@
 Wire Wire Line
 	4500 4900 4750 4900
-$Comp
-L C C9
-U 1 1 5B16F6A7
-P 4900 3800
-F 0 "C9" H 4925 3900 50  0000 L CNN
-F 1 "C" H 4925 3700 50  0000 L CNN
-F 2 "Capacitors_THT:CP_Radial_D10.0mm_P5.00mm" H 4938 3650 50  0001 C CNN
-F 3 "" H 4900 3800 50  0001 C CNN
-	1    4900 3800
-	1    0    0    -1
-$EndComp
 Wire Wire Line
 	5100 3650 5100 3600
@@
 	5100 3950 5100 4000
 Wire Wire Line
-	4900 3650 4900 3600
-Connection ~ 4900 3600
-Wire Wire Line
-	4900 3950 4650 3950
-Wire Wire Line
 	4650 3950 4650 4000
