File: Hardware/Elektrische_Komm.sch (KiCad schematic (older format))
At the start: 123 parts, among them J1 Conn_01x01, J2 Conn_01x01, J3 Conn_01x01, J4 Conn_01x04, J5 USB_OTG, J6 Conn_01x01, J7 Conn_01x01, Q1 CSD16556Q5B, Q10 BSR202NL6327HTSA1, Q11 BSR202NL6327HTSA1, Q12 BSR202NL6327HTSA1, Q13 BSR202NL6327HTSA1, Q14 BSR202NL6327HTSA1, Q2 CSD16556Q5B, Q3 CSD16556Q5B, Q4 CSD16556Q5B, Q5 CSD16556Q5B, Q6 CSD16556Q5B, Q7 BSR202NL6327HTSA1, Q8 BSR202NL6327HTSA1, Q9 BSR202NL6327HTSA1, SW1 SW_Push, SW2 SW_Push, U1 TS374IDT, U10 TPS561201, U12 STM32F413R(G-H)Tx_u, U2 UCC27710, U3 ACS723LLCTR, U4 UCC27710, U5 MCP6546, U6 UCC27710, U7 NC7WZ32, U8 74LVC2G02, Y1 24MHz

Commit message: ___________ < remodeled >  -----------       \                    / \  //\        \    |\___/|      /   \//  \\             /0  0  \__  /    //  | \ \            /     /  \/_/    //   |  \  \            @_^_@'/   \/_   //    |   \   \            //_^_/     \/_ //     |    \    \         ( //) |        \///      |     \     \       ( / /) _|_ /   )  //       |      \     _\     ( // /) '/,_ _ _/  ( ; -.    |    _ _\.-~        .-~~~^-.   (( / / )) ,-{        _      `-.|.-~-.           .~         `.  (( // / ))  '/\      /                 ~-. _ .-~      .-~^-.  \  (( /// ))      `.   {            }                   /      \  \   (( / ))     .----~-.\        \-'                 .~         \  `. \^-.              ///.----..>        \             _ -~             `.  ^-`  ^-_                ///-._ _ _ _ _ _ _}^ - - - - ~                     ~-- ,.-~                                                                   /.-~
Parts:
- removed U7: NC7WZ32, Housings_SSOP:VSSOP-8_2.3x2mm_Pitch0.5mm, symbol NC7WZ32
- added C14, C15, C9: C, Capacitors_SMD:C_1812, symbol C
- added C?: C, Capacitors_THT:CP_Radial_D10.0mm_P5.00mm, symbol C
- added R11, R12, R14, R15, R8: R, Resistors_SMD:R_0603, symbol R
- added unit 4 of U1
- added U7: 74HC32D, Housings_SSOP:TSSOP-14_4.4x5mm_Pitch0.65mm, symbol 74HC32D
Connections:
- net labels added: OR1, OVoltage
- net labels removed: Stop_Hardware
- wire segments 360 -> 388

Commit message: ______________________ < Layout überarbeitet >  ----------------------       \                    / \  //\        \    |\___/|      /   \//  \\             /0  0  \__  /    //  | \ \            /     /  \/_/    //   |  \  \            @_^_@'/   \/_   //    |   \   \            //_^_/     \/_ //     |    \    \         ( //) |        \///      |     \     \       ( / /) _|_ /   )  //       |      \     _\     ( // /) '/,_ _ _/  ( ; -.    |    _ _\.-~        .-~~~^-.   (( / / )) ,-{        _      `-.|.-~-.           .~         `.  (( // / ))  '/\      /                 ~-. _ .-~      .-~^-.  \  (( /// ))      `.   {            }                   /      \  \   (( / ))     .----~-.\        \-'                 .~         \  `. \^-.              ///.----..>        \             _ -~             `.  ^-`  ^-_                ///-._ _ _ _ _ _ _}^ - - - - ~                     ~-- ,.-~                                                                   /.-~
Parts:
- gave numbers to parts that had none: 1
Connections:
- net VCC: now also C6.1

Commit message: ________________ < Mounting Holes >  ----------------       \                    / \  //\        \    |\___/|      /   \//  \\             /0  0  \__  /    //  | \ \            /     /  \/_/    //   |  \  \            @_^_@'/   \/_   //    |   \   \            //_^_/     \/_ //     |    \    \         ( //) |        \///      |     \     \       ( / /) _|_ /   )  //       |      \     _\     ( // /) '/,_ _ _/  ( ; -.    |    _ _\.-~        .-~~~^-.   (( / / )) ,-{        _      `-.|.-~-.           .~         `.  (( // / ))  '/\      /                 ~-. _ .-~      .-~^-.  \  (( /// ))      `.   {            }                   /      \  \   (( / ))     .----~-.\        \-'                 .~         \  `. \^-.              ///.----..>        \             _ -~             `.  ^-`  ^-_                ///-._ _ _ _ _ _ _}^ - - - - ~                     ~-- ,.-~                                                                   /.-~
Parts:
- added J10, J11, J8, J9: Screw_Terminal_01x01, Mounting_Holes:MountingHole_3.2mm_M3_DIN965, symbol Screw_Terminal_01x01
- R8: value R -> 10k
Other:
- note added: "Befestigungslöcher"
Changed lines of the file:
@@
 P 10850 4800
 F 0 "R8" V 10930 4800 50  0000 C CNN
-F 1 "R" V 10850 4800 50  0000 C CNN
+F 1 "10k" V 10850 4800 50  0000 C CNN
 F 2 "Resistors_SMD:R_0603" V 10780 4800 50  0001 C CNN
 F 3 "" H 10850 4800 50  0001 C CNN
@@
 Wire Wire Line
 	4650 3600 4650 3650
+$Comp
+L Screw_Terminal_01x01 J8
+U 1 1 5B278AAC
+P 16550 6350
+F 0 "J8" H 16550 6450 50  0000 C CNN
+F 1 "Screw_Terminal_01x01" H 16550 6250 50  0000 C CNN
+F 2 "Mounting_Holes:MountingHole_3.2mm_M3_DIN965" H 16550 6350 50  0001 C CNN
+F 3 "" H 16550 6350 50  0001 C CNN
+	1    16550 6350
+	1    0    0    -1
+$EndComp
+$Comp
+L Screw_Terminal_01x01 J9
+U 1 1 5B279313
+P 17500 6350
+F 0 "J9" H 17500 6450 50  0000 C CNN
+F 1 "Screw_Terminal_01x01" H 17500 6250 50  0000 C CNN
+F 2 "Mounting_Holes:MountingHole_3.2mm_M3_DIN965" H 17500 6350 50  0001 C CNN
+F 3 "" H 17500 6350 50  0001 C CNN
+	1    17500 6350
+	1    0    0    -1
+$EndComp
+$Comp
+L Screw_Terminal_01x01 J11
+U 1 1 5B2794FE
+P 17500 6700
+F 0 "J11" H 17500 6800 50  0000 C CNN
+F 1 "Screw_Terminal_01x01" H 17500 6600 50  0000 C CNN
+F 2 "Mounting_Holes:MountingHole_3.2mm_M3_DIN965" H 17500 6700 50  0001 C CNN
+F 3 "" H 17500 6700 50  0001 C CNN
+	1    17500 6700
+	1    0    0    -1
+$EndComp
+$Comp
+L Screw_Terminal_01x01 J10
+U 1 1 5B2796D4
+P 16550 6700
+F 0 "J10" H 16550 6800 50  0000 C CNN
+F 1 "Screw_Terminal_01x01" H 16550 6600 50  0000 C CNN
+F 2 "Mounting_Holes:MountingHole_3.2mm_M3_DIN965" H 16550 6700 50  0001 C CNN
+F 3 "" H 16550 6700 50  0001 C CNN
+	1    16550 6700
+	1    0    0    -1
+$EndComp
+Text Notes 16250 7100 0    60   ~ 0
+Befestigungslöcher
 $EndSCHEMATC

Commit message: Board fertig
Parts:
- removed J11: Screw_Terminal_01x01, Mounting_Holes:MountingHole_3.2mm_M3_DIN965, symbol Screw_Terminal_01x01
- added J12, J13, J14: Conn_01x01, kicadBibs:Führungsloch, symbol Conn_01x01
Changed lines of the file:
@@
 	5400 2500 450  2500
 Wire Wire Line
-	1600 2250 1600 2100
+	1600 2100 1600 2250
 Wire Wire Line
 	3000 2100 3000 2250
@@
 Connection ~ 5600 2200
 Wire Wire Line
-	4500 2250 4500 2100
+	4500 2100 4500 2250
 Wire Wire Line
 	7300 2200 8050 2200
@@
 	11700 1500 12100 1500
 Wire Notes Line
-	11400 1850 12800 1850
-Wire Notes Line
-	12800 1850 12800 450
+	11400 1850 13150 1850
 Wire Wire Line
 	800  700  4500 700
@@
 $EndComp
 $Comp
-L Screw_Terminal_01x01 J11
-U 1 1 5B2794FE
-P 17500 6700
-F 0 "J11" H 17500 6800 50  0000 C CNN
-F 1 "Screw_Terminal_01x01" H 17500 6600 50  0000 C CNN
-F 2 "Mounting_Holes:MountingHole_3.2mm_M3_DIN965" H 17500 6700 50  0001 C CNN
-F 3 "" H 17500 6700 50  0001 C CNN
-	1    17500 6700
-	1    0    0    -1
-$EndComp
-$Comp
 L Screw_Terminal_01x01 J10
 U 1 1 5B2796D4
@@
 Text Notes 16250 7100 0    60   ~ 0
 Befestigungslöcher
+$Comp
+L Conn_01x01 J12
+U 1 1 5B2B78E1
+P 12800 900
+F 0 "J12" H 12800 1000 50  0000 C CNN
+F 1 "Conn_01x01" H 12800 800 50  0000 C CNN
+F 2 "kicadBibs:Führungsloch" H 12800 900 50  0001 C CNN
+F 3 "" H 12800 900 50  0001 C CNN
+	1    12800 900
+	1    0    0    -1
+$EndComp
+$Comp
+L Conn_01x01 J13
+U 1 1 5B2B7AC7
+P 12800 1200
+F 0 "J13" H 12800 1300 50  0000 C CNN
+F 1 "Conn_01x01" H 12800 1100 50  0000 C CNN
+F 2 "kicadBibs:Führungsloch" H 12800 1200 50  0001 C CNN
+F 3 "" H 12800 1200 50  0001 C CNN
+	1    12800 1200
+	1    0    0    -1
+$EndComp
+$Comp
+L Conn_01x01 J14
+U 1 1 5B2B7CB2
+P 12800 1500
+F 0 "J14" H 12800 1600 50  0000 C CNN
+F 1 "Conn_01x01" H 12800 1400 50  0000 C CNN
+F 2 "kicadBibs:Führungsloch" H 12800 1500 50  0001 C CNN
+F 3 "" H 12800 1500 50  0001 C CNN
+	1    12800 1500
+	1    0    0    -1
+$EndComp
+Wire Notes Line
+	13150 1850 13150 450
 $EndSCHEMATC

Commit message: _________________________ < Zener-Spannungsreferenz >  -------------------------       \                    / \  //\        \    |\___/|      /   \//  \\             /0  0  \__  /    //  | \ \            /     /  \/_/    //   |  \  \            @_^_@'/   \/_   //    |   \   \            //_^_/     \/_ //     |    \    \         ( //) |        \///      |     \     \       ( / /) _|_ /   )  //       |      \     _\     ( // /) '/,_ _ _/  ( ; -.    |    _ _\.-~        .-~~~^-.   (( / / )) ,-{        _      `-.|.-~-.           .~         `.  (( // / ))  '/\      /                 ~-. _ .-~      .-~^-.  \  (( /// ))      `.   {            }                   /      \  \   (( / ))     .----~-.\        \-'                 .~         \  `. \^-.              ///.----..>        \             _ -~             `.  ^-`  ^-_                ///-._ _ _ _ _ _ _}^ - - - - ~                     ~-- ,.-~                                                                   /.-~
Parts:
- removed R14: R, Resistors_SMD:R_0603, symbol R
- added D2: MM3Z5V6T1G, Diodes_SMD:D_SOD-323, symbol D_Zener
- C10, C3, C7: footprint Capacitors_SMD:C_0603 -> Capacitors_SMD:C_0805
- C13: footprint Capacitors_SMD:C_1206 -> Capacitors_SMD:C_0805
- R11: value R -> 9,4k
- R12: value R -> 523k
- R15, R16: value R -> 100k
- R35, R36, R37, R38, R39: value R -> 100
Connections:
- net GNDREF: now also D2.2 (A)
- net at R11.2, U1.10 (-): now also D2.1 (K)
Other:
- note added: "Laborklemmen"
- note added: "Überspannungsschutz"
Changed lines of the file:
@@
 F 0 "C3" H 5625 2550 50  0000 L CNN
 F 1 "47µ" H 5625 2350 50  0000 L CNN
-F 2 "Capacitors_SMD:C_0603" H 5638 2300 50  0001 C CNN
+F 2 "Capacitors_SMD:C_0805" H 5638 2300 50  0001 C CNN
 F 3 "" H 5600 2450 50  0001 C CNN
 	1    5600 2450
@@
 F 0 "C7" H 5675 4000 50  0000 L CNN
 F 1 "47µ" H 5675 3800 50  0000 L CNN
-F 2 "Capacitors_SMD:C_0603" H 5688 3750 50  0001 C CNN
+F 2 "Capacitors_SMD:C_0805" H 5688 3750 50  0001 C CNN
 F 3 "" H 5650 3900 50  0001 C CNN
 	1    5650 3900
@@
 F 0 "C10" H 5675 5400 50  0000 L CNN
 F 1 "47µ" H 5675 5200 50  0000 L CNN
-F 2 "Capacitors_SMD:C_0603" H 5688 5150 50  0001 C CNN
+F 2 "Capacitors_SMD:C_0805" H 5688 5150 50  0001 C CNN
 F 3 "" H 5650 5300 50  0001 C CNN
 	1    5650 5300
@@
 P 5100 3800
 F 0 "R16" V 5180 3800 50  0000 C CNN
-F 1 "R" V 5100 3800 50  0000 C CNN
+F 1 "100k" V 5100 3800 50  0000 C CNN
 F 2 "Resistors_SMD:R_0603" V 5030 3800 50  0001 C CNN
 F 3 "" H 5100 3800 50  0001 C CNN
@@
 P 8150 11650
 F 0 "R36" V 8230 11650 50  0000 C CNN
-F 1 "R" V 8150 11650 50  0000 C CNN
+F 1 "100" V 8150 11650 50  0000 C CNN
 F 2 "Resistors_SMD:R_0603" V 8080 11650 50  0001 C CNN
 F 3 "" H 8150 11650 50  0001 C CNN
@@
 P 7350 11650
 F 0 "R35" V 7430 11650 50  0000 C CNN
-F 1 "R" V 7350 11650 50  0000 C CNN
+F 1 "100" V 7350 11650 50  0000 C CNN
 F 2 "Resistors_SMD:R_0603" V 7280 11650 50  0001 C CNN
 F 3 "" H 7350 11650 50  0001 C CNN
@@
 P 8900 11650
 F 0 "R37" V 8980 11650 50  0000 C CNN
-F 1 "R" V 8900 11650 50  0000 C CNN
+F 1 "100" V 8900 11650 50  0000 C CNN
 F 2 "Resistors_SMD:R_0603" V 8830 11650 50  0001 C CNN
 F 3 "" H 8900 11650 50  0001 C CNN
@@
 P 9650 11650
 F 0 "R38" V 9730 11650 50  0000 C CNN
-F 1 "R" V 9650 11650 50  0000 C CNN
+F 1 "100" V 9650 11650 50  0000 C CNN
 F 2 "Resistors_SMD:R_0603" V 9580 11650 50  0001 C CNN
 F 3 "" H 9650 11650 50  0001 C CNN
@@
 F 0 "C13" H 14975 7050 50  0000 L CNN
 F 1 "47µ" H 14975 6850 50  0000 L CNN
-F 2 "Capacitors_SMD:C_1206" H 14988 6800 50  0001 C CNN
+F 2 "Capacitors_SMD:C_0805" H 14988 6800 50  0001 C CNN
 F 3 "" H 14950 6950 50  0001 C CNN
 	1    14950 6950
@@
 P 10300 11700
 F 0 "R39" V 10380 11700 50  0000 C CNN
-F 1 "R" V 10300 11700 50  0000 C CNN
+F 1 "100" V 10300 11700 50  0000 C CNN
 F 2 "Resistors_SMD:R_0603" V 10230 11700 50  0001 C CNN
 F 3 "" H 10300 11700 50  0001 C CNN
@@
 P 8800 5000
 F 0 "R11" V 8880 5000 50  0000 C CNN
-F 1 "R" V 8800 5000 50  0000 C CNN
+F 1 "9,4k" V 8800 5000 50  0000 C CNN
 F 2 "Resistors_SMD:R_0603" V 8730 5000 50  0001 C CNN
 F 3 "" H 8800 5000 50  0001 C CNN
@@
 P 9200 5000
 F 0 "R12" V 9280 5000 50  0000 C CNN
-F 1 "R" V 9200 5000 50  0000 C CNN
+F 1 "523k" V 9200 5000 50  0000 C CNN
 F 2 "Resistors_SMD:R_0603" V 9130 5000 50  0001 C CNN
 F 3 "" H 9200 5000 50  0001 C CNN
@@
 P 9200 5500
 F 0 "R15" V 9280 5500 50  0000 C CNN
-F 1 "R" V 9200 5500 50  0000 C CNN
+F 1 "100k" V 9200 5500 50  0000 C CNN
 F 2 "Resistors_SMD:R_0603" V 9130 5500 50  0001 C CNN
 F 3 "" H 9200 5500 50  0001 C CNN
@@
 $EndComp
 $Comp
-L R R14
-U 1 1 5B240686
-P 8800 5500
-F 0 "R14" V 8880 5500 50  0000 C CNN
-F 1 "R" V 8800 5500 50  0000 C CNN
-F 2 "Resistors_SMD:R_0603" V 8730 5500 50  0001 C CNN
-F 3 "" H 8800 5500 50  0001 C CNN
-	1    8800 5500
-	1    0    0    -1
-$EndComp
-$Comp
 L GNDREF #PWR075
 U 1 1 5B2407BE
@@
 	8800 5150 8800 5350
 Wire Wire Line
-	9800 5200 8800 5200
-Connection ~ 8800 5200
-Wire Wire Line
-	9800 4900 9550 4900
-Wire Wire Line
-	9550 4900 9550 5250
-Wire Wire Line
-	9550 5250 9200 5250
-Connection ~ 9200 5250
+	9450 4900 9800 4900
 Wire Wire Line
 	10850 4950 10850 5050
@@
 Wire Notes Line
 	13150 1850 13150 450
+Text Notes 10350 5900 0    60   ~ 0
+Überspannungsschutz
+$Comp
+L D_Zener D2
+U 1 1 5B2E838B
+P 8800 5500
+F 0 "D2" H 8800 5600 50  0000 C CNN
+F 1 "MM3Z5V6T1G" H 8800 5400 50  0000 C CNN
+F 2 "Diodes_SMD:D_SOD-323" H 8800 5500 50  0001 C CNN
+F 3 "" H 8800 5500 50  0001 C CNN
+	1    8800 5500
+	0    1    1    0
+$EndComp
+Wire Wire Line
+	9800 5200 9650 5200
+Wire Wire Line
+	9650 5200 9650 5300
+Wire Wire Line
+	9650 5300 8800 5300
+Connection ~ 8800 5300
+Wire Wire Line
+	9450 4900 9450 5200
+Wire Wire Line
+	9450 5200 9200 5200
+Connection ~ 9200 5200
+Text Notes 4550 5850 0    60   ~ 0
+Laborklemmen
 $EndSCHEMATC

Commit message: ________________________ < Gerber-Files geplottet >  ------------------------       \                    / \  //\        \    |\___/|      /   \//  \\             /0  0  \__  /    //  | \ \            /     /  \/_/    //   |  \  \            @_^_@'/   \/_   //    |   \   \            //_^_/     \/_ //     |    \    \         ( //) |        \///      |     \     \       ( / /) _|_ /   )  //       |      \     _\     ( // /) '/,_ _ _/  ( ; -.    |    _ _\.-~        .-~~~^-.   (( / / )) ,-{        _      `-.|.-~-.           .~         `.  (( // / ))  '/\      /                 ~-. _ .-~      .-~^-.  \  (( /// ))      `.   {            }                   /      \  \   (( / ))     .----~-.\        \-'                 .~         \  `. \^-.              ///.----..>        \             _ -~             `.  ^-`  ^-_                ///-._ _ _ _ _ _ _}^ - - - - ~                     ~-- ,.-~                                                                   /.-~
Parts:
- added R14: 1k, Resistors_SMD:R_0603, symbol R
- added SW3: SW_Push, kicadBibs:Switch, symbol SW_Push
- added TP26: TEST, Pin_Headers:Pin_Header_Straight_1x01_Pitch1.00mm, symbol TEST
Connections:
- net +3V3: now also R14.1
- net GNDREF: now also SW3.2
- net Meas_out: now also TP26.1
- net StopButton: now reaches U12.52 (PC11/ADC1_EXTI11/DFSDM2_DATIN5/FSMC_D2/FSMC_DA2/I2S3_ext_SD/QUADSPI_BK2_NCS/SDIO_D3/SPI3_MISO/UART4_RX/USART3_RX)
- net StopButton: now also R14.2, SW3.1
Other:
- note added: "Manueller Eingriff"
Changed lines of the file:
@@
 	6600 14400 5850 14400
 Connection ~ 5850 14400
-Wire Notes Line
-	6700 13050 6700 16100
 Wire Wire Line
 	900  6550 1600 6550
@@
 	1    0    0    -1
 $EndComp
-Text Notes 16250 7100 0    60   ~ 0
+Text Notes 16250 7100 0    118  ~ 0
 Befestigungslöcher
 $Comp
@@
 Text Notes 4550 5850 0    60   ~ 0
 Laborklemmen
+$Comp
+L TEST TP26
+U 1 1 5B338CBE
+P 3600 14950
+F 0 "TP26" H 3600 15250 50  0000 C BNN
+F 1 "TEST" H 3600 15200 50  0000 C CNN
+F 2 "Pin_Headers:Pin_Header_Straight_1x01_Pitch1.00mm" H 3600 14950 50  0001 C CNN
+F 3 "" H 3600 14950 50  0001 C CNN
+	1    3600 14950
+	0    -1   -1   0
+$EndComp
+Text Label 3600 14950 0    60   ~ 0
+Meas_out
+$Comp
+L R R14
+U 1 1 5B34FC72
+P 7200 14050
+F 0 "R14" V 7280 14050 50  0000 C CNN
+F 1 "1k" V 7200 14050 50  0000 C CNN
+F 2 "Resistors_SMD:R_0603" V 7130 14050 50  0001 C CNN
+F 3 "" H 7200 14050 50  0001 C CNN
+	1    7200 14050
+	1    0    0    -1
+$EndComp
+$Comp
+L +3.3V #PWR078
+U 1 1 5B34FC78
+P 7200 13750
+F 0 "#PWR078" H 7200 13600 50  0001 C CNN
+F 1 "+3.3V" H 7200 13890 50  0000 C CNN
+F 2 "" H 7200 13750 50  0001 C CNN
+F 3 "" H 7200 13750 50  0001 C CNN
+	1    7200 13750
+	1    0    0    -1
+$EndComp
+$Comp
+L SW_Push SW3
+U 1 1 5B34FC7E
+P 7200 14550
+F 0 "SW3" H 7250 14650 50  0000 L CNN
+F 1 "SW_Push" H 7200 14490 50  0000 C CNN
+F 2 "kicadBibs:Switch" H 7200 14750 50  0001 C CNN
+F 3 "" H 7200 14750 50  0001 C CNN
+	1    7200 14550
+	0    1    1    0
+$EndComp
+$Comp
+L GNDREF #PWR079
+U 1 1 5B34FC84
+P 7200 14950
+F 0 "#PWR079" H 7200 14700 50  0001 C CNN
+F 1 "GNDREF" H 7200 14800 50  0000 C CNN
+F 2 "" H 7200 14950 50  0001 C CNN
+F 3 "" H 7200 14950 50  0001 C CNN
+	1    7200 14950
+	1    0    0    -1
+$EndComp
+Wire Wire Line
+	7200 13750 7200 13900
+Wire Wire Line
+	7200 14950 7200 14750
+Wire Wire Line
+	7200 14200 7200 14350
+Wire Wire Line
+	7450 14250 7200 14250
+Connection ~ 7200 14250
+Text Label 16800 10300 0    60   ~ 0
+StopButton
+Wire Wire Line
+	16800 10300 16600 10300
+Text Label 7450 14250 0    60   ~ 0
+StopButton
+Wire Notes Line
+	8000 13050 8000 16100
+Text Notes 6200 15900 0    118  ~ 0
+Manueller Eingriff
 $EndSCHEMATC

Commit message: __________________________ < Messstation hinzugefügt >  --------------------------       \                    / \  //\        \    |\___/|      /   \//  \\             /0  0  \__  /    //  | \ \            /     /  \/_/    //   |  \  \            @_^_@'/   \/_   //    |   \   \            //_^_/     \/_ //     |    \    \         ( //) |        \///      |     \     \       ( / /) _|_ /   )  //       |      \     _\     ( // /) '/,_ _ _/  ( ; -.    |    _ _\.-~        .-~~~^-.   (( / / )) ,-{        _      `-.|.-~-.           .~         `.  (( // / ))  '/\      /                 ~-. _ .-~      .-~^-.  \  (( /// ))      `.   {            }                   /      \  \   (( / ))     .----~-.\        \-'                 .~         \  `. \^-.              ///.----..>        \             _ -~             `.  ^-`  ^-_                ///-._ _ _ _ _ _ _}^ - - - - ~                     ~-- ,.-~                                                                   /.-~
Parts:
- added D11, D12, D13, D14: BZT52-C3V0X, Diodes_SMD:D_SOD-123, symbol D_Zener_ALT
- added R20, R21, R28, R32: 4M, Resistors_SMD:R_0603, symbol R
- added R33, R34, R40, R43: 1M, Resistors_SMD:R_0603, symbol R
Connections:
- net A: now also R32.1
- net B: now also R21.1
- net C: now also R20.1
- net GNDREF: now also D11.2 (A), D12.2 (A), D13.2 (A), D14.2 (A), R33.2, R34.2, R40.2, R43.2
- net Sternpunkt_virtuell: now also R28.1
- net Me_B: now reaches U12.10 (PC2/ADC1_IN12/DFSDM1_CKOUT/DFSDM2_DATIN7/FSMC_NWE/I2S2_ext_SD/LPTIM1_IN2/SAI1_SCK_B/SPI2_MISO)
- net Me_B: now also D12.1 (K), R21.2, R34.1
- net Me_C: now reaches U12.11 (PC3/ADC1_IN13/DFSDM2_CKIN7/FSMC_A0/I2S2_SD/LPTIM1_ETR/SAI1_FS_B/SPI2_MOSI)
- net Me_C: now also D11.1 (K), R20.2, R33.1
- net Me_A: now reaches U12.8 (PC0/ADC1_IN10/DFSDM2_CKIN4/LPTIM1_IN1/SAI1_MCLK_B/SYS_WKUP2)
- net Me_A: now also D14.1 (K), R32.2, R43.1
- net Me_VS: now reaches U12.9 (PC1/ADC1_IN11/DFSDM2_DATIN4/LPTIM1_OUT/SAI1_SD_B/SYS_WKUP3)
- net Me_VS: now also D13.1 (K), R28.2, R40.1
Other:
- note added: "Motormessung"
