File: Hardware/Elektrische_Komm.kicad_pcb (KiCad board)
At the start: 4 copper layers, 123 parts, among them J1 Conn_01x01, J2 Conn_01x01, J3 Conn_01x01, J4 Conn_01x04, J5 USB_OTG, Q1 BSZ014NE2LS5IF, Q10 BSR202NL6327HTSA1, Q11 BSR202NL6327HTSA1, Q12 BSR202NL6327HTSA1, Q13 BSR202NL6327HTSA1, Q14 BSR202NL6327HTSA1, Q2 BSZ014NE2LS5IF, Q3 BSZ014NE2LS5IF, Q4 BSZ014NE2LS5IF, Q5 BSZ014NE2LS5IF, Q6 BSZ014NE2LS5IF, Q7 BSR202NL6327HTSA1, Q8 BSR202NL6327HTSA1, Q9 BSR202NL6327HTSA1, SW1 SW_Push, SW2 SW_Push, U1 TS374IDT, U10 TPS561201, U11 TLC352, U12 STM32F413R(G-H)Tx_u, U2 UCC27710, U3 ACS723LLCTR, U4 UCC27710, U6 UCC27710, U7 74HC32D, U8 74LVC2G02, Y1 24MHz

Commit message: _______________________ < Layout weitergeführt >  -----------------------       \                    / \  //\        \    |\___/|      /   \//  \\             /0  0  \__  /    //  | \ \            /     /  \/_/    //   |  \  \            @_^_@'/   \/_   //    |   \   \            //_^_/     \/_ //     |    \    \         ( //) |        \///      |     \     \       ( / /) _|_ /   )  //       |      \     _\     ( // /) '/,_ _ _/  ( ; -.    |    _ _\.-~        .-~~~^-.   (( / / )) ,-{        _      `-.|.-~-.           .~         `.  (( // / ))  '/\      /                 ~-. _ .-~      .-~^-.  \  (( /// ))      `.   {            }                   /      \  \   (( / ))     .----~-.\        \-'                 .~         \  `. \^-.              ///.----..>        \             _ -~             `.  ^-`  ^-_                ///-._ _ _ _ _ _ _}^ - - - - ~                     ~-- ,.-~                                                                   /.-~
Parts:
- D1, D3, D5: footprint kicadBibs:SOD-123W -> Diodes_SMD:D_SOD-123F
- moved C16 48.6 mm to (220.2, 42.5)
- moved C12 47.9 mm to (214.7, 38.4), turned to 90 degrees
- moved R24 46.0 mm to (212.6, 39.2), turned to 90 degrees
- moved R26 45.0 mm to (210.9, 39.2), turned to 270 degrees
- moved L1 44.7 mm to (214.6, 42.4), turned to 180 degrees
- moved C13 42.5 mm to (214.7, 45.5)
- moved U10 24.6 mm to (217.5, 38.5)
- moved R7 18.7 mm to (255.7, 70.5), turned to 270 degrees
- moved R10 18.3 mm to (255.8, 65.1), turned to 270 degrees
- moved R2 16.2 mm to (253.4, 71.8), turned to 0 degrees
- moved C1 15.5 mm to (251.4, 73.9), turned to 270 degrees
- moved SW2 11.1 mm to (197.7, 35.2), turned to 90 degrees
- moved U1 10.0 mm to (250.1, 67.1), turned to 90 degrees
- moved C3 8.88 mm to (224.7, 54.7)
- moved R6 8.88 mm to (224.7, 50.7)
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Connections:
- net /DCDC_EN renamed /VCC
- C2 pad 2: /A_conn -> /A
- C5 pad 2: /B_conn -> /B
- TP3 pad 1: /B_conn -> (no net)
- U1 pad 4: /A_conn -> /A
- U1 pad 6: /B_conn -> /B
- U12 pad 41: /Bemf_A -> /Bemf_C
- U12 pad 43: /Bemf_C -> /Bemf_A
- U2 pad 6: /A_conn -> /A
- U4 pad 6: /B_conn -> /B
Routing:
- net /Bemf_A: track 2.03 -> 69.6 mm, vias 0 -> 1
- net /Bemf_B: track 1.86 -> 59.7 mm, vias 0 -> 1
- net /Over_curr: track 32.4 -> 90.0 mm, vias 0 -> 1
- net /Bemf_C: track 1.87 -> 54.0 mm, vias 0 -> 3
- net /A: track 10.0 -> 56.8 mm
- net /B: track 4.84 -> 32.9 mm
- net /HI_A_F: track 3.38 -> 26.9 mm, vias 0 -> 1
- net /HI_C_F: track 3.90 -> 22.4 mm, vias 0 -> 1
- net /D+: track 0.00 -> 13.5 mm
- net /D-: track 0.00 -> 13.5 mm
- net /A_conn: track 5.83 -> 0.00 mm
- net /C: track 34.7 -> 39.0 mm
- net /HI_B_F: track 3.69 -> 7.77 mm, vias 0 -> 1
- net Net-(D9-Pad1): track 2.86 -> 5.39 mm
- net /Freigabe_button: track 15.3 -> 17.6 mm
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- removed copper zone on B.Cu, net /Sternpunkt_virtuell
Other:
- net class Boost-Caps added: clearance 0.2, trace_width 0.5, via_dia 1.2, via_drill 0.8

Commit message: _______________________________ < K_ind Berechnung hinzugefügt >  -------------------------------       \                    / \  //\        \    |\___/|      /   \//  \\             /0  0  \__  /    //  | \ \            /     /  \/_/    //   |  \  \            @_^_@'/   \/_   //    |   \   \            //_^_/     \/_ //     |    \    \         ( //) |        \///      |     \     \       ( / /) _|_ /   )  //       |      \     _\     ( // /) '/,_ _ _/  ( ; -.    |    _ _\.-~        .-~~~^-.   (( / / )) ,-{        _      `-.|.-~-.           .~         `.  (( // / ))  '/\      /                 ~-. _ .-~      .-~^-.  \  (( /// ))      `.   {            }                   /      \  \   (( / ))     .----~-.\        \-'                 .~         \  `. \^-.              ///.----..>        \             _ -~             `.  ^-`  ^-_                ///-._ _ _ _ _ _ _}^ - - - - ~                     ~-- ,.-~                                                                   /.-~
Parts:
- moved D10 50.9 mm to (252.0, 43.4)
- moved R39 50.9 mm to (252.0, 39.7)
- moved R50 2.83 mm to (203.1, 43.4), turned to 0 degrees
- moved R51 2.80 mm to (205.9, 43.4), turned to 0 degrees
Routing:
- net /Curr_direct_A: track 22.8 -> 61.4 mm, vias 2 -> 4
- net /LI_C: track 0.00 -> 34.0 mm, vias 0 -> 3
- net /LI_A: track 0.00 -> 25.6 mm, vias 0 -> 2
- net /LI_B: track 0.00 -> 19.4 mm, vias 0 -> 3
- net /Freigabe_button: track 17.6 -> 21.6 mm

Commit message: ______________________ < Layout weitergemacht >  ----------------------       \                    / \  //\        \    |\___/|      /   \//  \\             /0  0  \__  /    //  | \ \            /     /  \/_/    //   |  \  \            @_^_@'/   \/_   //    |   \   \            //_^_/     \/_ //     |    \    \         ( //) |        \///      |     \     \       ( / /) _|_ /   )  //       |      \     _\     ( // /) '/,_ _ _/  ( ; -.    |    _ _\.-~        .-~~~^-.   (( / / )) ,-{        _      `-.|.-~-.           .~         `.  (( // / ))  '/\      /                 ~-. _ .-~      .-~^-.  \  (( /// ))      `.   {            }                   /      \  \   (( / ))     .----~-.\        \-'                 .~         \  `. \^-.              ///.----..>        \             _ -~             `.  ^-`  ^-_                ///-._ _ _ _ _ _ _}^ - - - - ~                     ~-- ,.-~                                                                   /.-~
Parts:
- R18, R5, R9: footprint Resistors_SMD:R_0603 -> Resistors_SMD:R_1210
- moved TP14 76.6 mm to (251.9, 38.5)
- moved TP15 75.7 mm to (251.9, 40.4)
- moved TP25 63.9 mm to (243.1, 41.8)
- moved TP24 62.3 mm to (241.6, 41.8)
- moved TP23 60.8 mm to (240.1, 41.8)
- moved TP1 30.5 mm to (204.0, 52.1)
- moved R5 11.6 mm to (216.1, 61.6), turned to 0 degrees
- moved R39 7.10 mm to (258.5, 36.9)
- moved D10 7.10 mm to (258.5, 40.6)
- moved D1 3.46 mm to (214.8, 57.5), turned to 270 degrees
- moved R9 3.06 mm to (235.4, 51.6)
- moved R18 3.01 mm to (251.9, 51.6)
- moved R30 1.56 mm to (241.6, 44.0)
- moved R31 1.56 mm to (243.1, 44.0)
- moved R29 1.56 mm to (240.0, 44.0)
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Connections:
- R18 pad 2: +15V -> /VCC
- R5 pad 2: +15V -> /VCC
- R9 pad 2: +15V -> /VCC
- TP2 pad 1: /A_conn -> /A
- TP3 pad 1: (no net) -> /B
- U12 pad 10: /C -> (no net)
- U12 pad 11: /Sternpunkt_virtuell -> (no net)
- U12 pad 8: /A -> (no net)
- U12 pad 9: /B -> (no net)
Routing:
- net /DAC1: track 0.00 -> 16.1 mm, vias 0 -> 2
- net /DAC2: track 0.00 -> 14.6 mm, vias 0 -> 2
- net Net-(R24-Pad2): track 0.00 -> 11.0 mm
- net /DCDC_sw: track 0.00 -> 7.63 mm
- net /Curr_direct_A: track 61.4 -> 68.4 mm
- net /VCC: track 3.43 -> 9.63 mm
- net +3V3: track 20.6 -> 26.0 mm
- net Net-(C8-Pad1): track 0.00 -> 4.60 mm
- net Net-(C5-Pad1): track 0.00 -> 4.07 mm
- net Net-(D5-Pad2): track 0.00 -> 3.31 mm
- net Net-(D3-Pad2): track 0.00 -> 3.31 mm
- net Net-(C12-Pad2): track 0.00 -> 1.92 mm
- net /HI_A: track 1.69 -> 3.17 mm
- net /HI_C: track 2.44 -> 3.91 mm
- net /HI_B: track 2.50 -> 3.97 mm
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- added copper zone on F.Cu, net +3V3
- added copper zone on F.Cu, net /DCDC_sw
- added copper zone on B.Cu, net /Sternpunkt_virtuell
- added copper zone on B.Cu, net Net-(C5-Pad1)
- added copper zone on B.Cu, net Net-(C8-Pad1)
- added copper zone on B.Cu, net Net-(D1-Pad2)
- added copper zone on B.Cu, net Net-(D3-Pad2)
- added copper zone on B.Cu, net Net-(D5-Pad2)
- removed copper zone on B.Cu, net /A_conn
