File: Hardware/Elektrische_Komm.kicad_pcb (KiCad board)
At the start: 4 copper layers, 123 parts, among them J1 Conn_01x01, J2 Conn_01x01, J3 Conn_01x01, J4 Conn_01x04, J5 USB_OTG, Q1 BSZ014NE2LS5IF, Q10 BSR202NL6327HTSA1, Q11 BSR202NL6327HTSA1, Q12 BSR202NL6327HTSA1, Q13 BSR202NL6327HTSA1, Q14 BSR202NL6327HTSA1, Q2 BSZ014NE2LS5IF, Q3 BSZ014NE2LS5IF, Q4 BSZ014NE2LS5IF, Q5 BSZ014NE2LS5IF, Q6 BSZ014NE2LS5IF, Q7 BSR202NL6327HTSA1, Q8 BSR202NL6327HTSA1, Q9 BSR202NL6327HTSA1, SW1 SW_Push, SW2 SW_Push, U1 TS374IDT, U10 TPS561201, U11 TLC352, U12 STM32F413R(G-H)Tx_u, U2 UCC27710, U3 ACS723LLCTR, U4 UCC27710, U6 UCC27710, U7 74HC32D, U8 74LVC2G02, Y1 24MHz

Commit message: ___________________ < MOSFETS geändert >  -------------------       \                    / \  //\        \    |\___/|      /   \//  \\             /0  0  \__  /    //  | \ \            /     /  \/_/    //   |  \  \            @_^_@'/   \/_   //    |   \   \            //_^_/     \/_ //     |    \    \         ( //) |        \///      |     \     \       ( / /) _|_ /   )  //       |      \     _\     ( // /) '/,_ _ _/  ( ; -.    |    _ _\.-~        .-~~~^-.   (( / / )) ,-{        _      `-.|.-~-.           .~         `.  (( // / ))  '/\      /                 ~-. _ .-~      .-~^-.  \  (( /// ))      `.   {            }                   /      \  \   (( / ))     .----~-.\        \-'                 .~         \  `. \^-.              ///.----..>        \             _ -~             `.  ^-`  ^-_                ///-._ _ _ _ _ _ _}^ - - - - ~                     ~-- ,.-~                                                                   /.-~
Parts:
- removed R28: 10k, Resistors_SMD:R_0603
- removed R50, R51: R, Resistors_SMD:R_0603
- removed U11: TLC352, Housings_SSOP:TSSOP-8_4.4x3mm_Pitch0.65mm
- added U5: MCP6546, TO_SOT_Packages_SMD:SOT-23-5, F.Cu at (206.5, 42.8)
- Q1, Q2, Q3, Q4, Q5, Q6: value BSZ014NE2LS5IF -> CSD16556Q5B; footprint kicadBibs:SON65P330X330X110-8N -> kicadBibs:SON5x6
- U7: value 74HC32D -> NC7WZ32; footprint Housings_SSOP:TSSOP-14_4.4x5mm_Pitch0.65mm -> Housings_SSOP:VSSOP-8_2.3x2mm_Pitch0.5mm
- moved TP10 81.8 mm to (264.6, 56.6)
- moved TP8 65.5 mm to (247.6, 56.4)
- moved TP6 46.3 mm to (227.0, 56.4)
- moved R22 12.8 mm to (204.9, 45.7), turned to 0 degrees
- moved R42 12.4 mm to (201.7, 36.7)
- moved R25 10.7 mm to (207.9, 39.6), turned to 0 degrees
- moved R27 9.91 mm to (209.7, 27.9)
- moved SW2 9.89 mm to (201.9, 26.2), turned to 270 degrees
- moved R23 8.35 mm to (207.9, 38.0)
- moved U7 8.12 mm to (206.8, 33.8), turned to 90 degrees
- moved Q6 7.69 mm to (261.0, 70.7), turned to 270 degrees
- moved Q4 7.65 mm to (221.0, 70.7), turned to 270 degrees
- moved Q5 7.64 mm to (241.0, 70.7), turned to 270 degrees
- moved C11 7.39 mm to (204.2, 33.7), turned to 270 degrees
- moved D6 6.67 mm to (221.8, 26.4)
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Connections:
- R22 pad 2: Net-(R22-Pad2) -> /Stop_Hardware
- U7 pad 1: /OR1 -> /Stop_Hardware
- U7 pad 3: /Stop -> Net-(R27-Pad2)
- U7 pad 4: (no net) -> GNDREF
- U7 pad 5: (no net) -> /Freigabe_button
- U7 pad 6: (no net) -> /Freigabe_MCU
- U7 pad 7: GNDREF -> /Stop
- U7 pad 8: Net-(R27-Pad2) -> +3V3
Routing:
- net Net-(R28-Pad2): track 17.8 -> 0.00 mm
- net /Curr_direct_A: track 68.4 -> 50.7 mm, vias 4 -> 2
- net /HO_A: track 0.00 -> 14.1 mm, vias 0 -> 1
- net /HO_B: track 0.00 -> 13.8 mm, vias 0 -> 1
- net Net-(R22-Pad2): track 12.0 -> 0.00 mm
- net /Stop_Hardware: track 0.00 -> 11.4 mm
- net /HO_C: track 0.00 -> 11.1 mm, vias 0 -> 1
- net Net-(R27-Pad2): track 1.86 -> 11.5 mm
- net /OR1: track 6.71 -> 0.00 mm
- net Net-(R50-Pad2): track 5.72 -> 0.00 mm
- net /Freigabe_button: track 21.6 -> 15.9 mm
- net /freigegeben: track 41.1 -> 36.0 mm
- net /Bemf_B: track 59.7 -> 55.2 mm
- net /C: track 39.6 -> 35.2 mm
- net /Bemf_C: track 54.0 -> 50.6 mm
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- added copper zone on F.Cu, net /A
- added copper zone on F.Cu, net /B
- added copper zone on F.Cu, net /C
- added copper zone on F.Cu, net /Meas_out
- added copper zone on F.Cu, net GNDREF

Commit message: _____________________ < BW_SEL hinzugefügt >  ---------------------       \                    / \  //\        \    |\___/|      /   \//  \\             /0  0  \__  /    //  | \ \            /     /  \/_/    //   |  \  \            @_^_@'/   \/_   //    |   \   \            //_^_/     \/_ //     |    \    \         ( //) |        \///      |     \     \       ( / /) _|_ /   )  //       |      \     _\     ( // /) '/,_ _ _/  ( ; -.    |    _ _\.-~        .-~~~^-.   (( / / )) ,-{        _      `-.|.-~-.           .~         `.  (( // / ))  '/\      /                 ~-. _ .-~      .-~^-.  \  (( /// ))      `.   {            }                   /      \  \   (( / ))     .----~-.\        \-'                 .~         \  `. \^-.              ///.----..>        \             _ -~             `.  ^-`  ^-_                ///-._ _ _ _ _ _ _}^ - - - - ~                     ~-- ,.-~                                                                   /.-~
Parts:
- moved TP2 87.1 mm to (264.2, 39.5)
- moved TP3 85.2 mm to (264.2, 44.3)
- moved TP5 84.0 mm to (264.2, 47.8)
- moved TP11 79.9 mm to (265.0, 73.4)
- moved TP22 72.8 mm to (252.1, 43.1)
- moved TP12 60.2 mm to (235.8, 43.7)
- moved TP9 60.0 mm to (245.0, 73.4)
- moved TP4 57.7 mm to (232.9, 43.7)
- moved TP7 40.0 mm to (225.0, 73.4)
- moved TP21 28.3 mm to (210.7, 64.0)
- moved R16 25.9 mm to (207.5, 63.1), turned to 270 degrees
- moved D10 14.3 mm to (255.5, 26.5), turned to 180 degrees
- moved R39 12.2 mm to (252.0, 26.5), turned to 0 degrees
Connections:
- TP2 pad 1: /A -> /Bemf_A
- TP3 pad 1: /B -> /Bemf_B
- TP5 pad 1: /C -> /Bemf_C
- U12 pad 17: (no net) -> /BW_SEL
- U3 pad 6: GNDREF -> /BW_SEL
Routing:
- net /BW_SEL: track 0.00 -> 37.5 mm
- net /Sternpunkt_virtuell: track 48.5 -> 70.4 mm, vias 0 -> 2
- net /Freigabe_button: track 15.9 -> 23.9 mm
- net GNDREF: track 1.27 -> 6.92 mm, vias 0 -> 5
- net /Bemf_A: track 66.9 -> 71.1 mm
- net /LI_C: track 34.7 -> 38.1 mm
- net /Bemf_C: track 50.6 -> 53.1 mm
- net /LO_C: track 0.00 -> 2.11 mm
- net /LO_B: track 0.00 -> 2.11 mm
- net /LO_A: track 0.00 -> 2.11 mm
- net /LI_A: track 25.6 -> 27.5 mm
- net /LI_B: track 19.4 -> 20.5 mm
- removed copper zone on F.Cu, net Net-(C21-Pad2)
Other:
- board text added: "BemfA"
- board text added: "BemfB"
- board text added: "BemfC"
- board text added: "CLK"
- board text added: "DAC1"
- board text added: "DAC2"
- board text added: "HO_A"
- board text added: "HO_B"
- board text added: "HO_C"
- board text added: "LI_A"
- board text added: "LI_B"
- board text added: "LI_C"
- board text added: "LO_A"
- board text added: "LO_B"
- board text added: "LO_C"
- board text added: "Motorstrom"
- board text added: "Sternpunkt"

Commit message: _________________ < Planes erledigt >  -----------------       \                    / \  //\        \    |\___/|      /   \//  \\             /0  0  \__  /    //  | \ \            /     /  \/_/    //   |  \  \            @_^_@'/   \/_   //    |   \   \            //_^_/     \/_ //     |    \    \         ( //) |        \///      |     \     \       ( / /) _|_ /   )  //       |      \     _\     ( // /) '/,_ _ _/  ( ; -.    |    _ _\.-~        .-~~~^-.   (( / / )) ,-{        _      `-.|.-~-.           .~         `.  (( // / ))  '/\      /                 ~-. _ .-~      .-~^-.  \  (( /// ))      `.   {            }                   /      \  \   (( / ))     .----~-.\        \-'                 .~         \  `. \^-.              ///.----..>        \             _ -~             `.  ^-`  ^-_                ///-._ _ _ _ _ _ _}^ - - - - ~                     ~-- ,.-~                                                                   /.-~
Parts:
- added C6: C, Capacitors_THT:CP_Radial_D10.0mm_P5.00mm, F.Cu at (197.0, 60.0)
- added C9: C, Capacitors_THT:CP_Radial_D10.0mm_P5.00mm, F.Cu at (197.0, 71.5)
- added J6: Conn_01x01, kicadBibs:Laborbuchse, F.Cu at (187.0, 51.5)
- added J7: Conn_01x01, kicadBibs:Laborbuchse, F.Cu at (187.0, 66.0)
- L1: footprint kicadBibs:NLCV32T-3R3M-EF -> kicadBibs:SRN3015-3R3M
- moved TP20 89.5 mm to (259.7, 26.5)
- moved TP13 81.3 mm to (251.2, 28.7)
- moved TP19 54.8 mm to (221.7, 35.3)
- moved TP16 31.4 mm to (209.4, 56.3)
- moved TP17 27.1 mm to (212.2, 75.1)
Connections:
- C1 pad 1: (no net) -> /Vin
Routing:
- net /LO_A: track 2.11 -> 21.3 mm, vias 0 -> 2
- net /LO_C: track 2.11 -> 20.7 mm, vias 0 -> 1
- net /LO_B: track 2.11 -> 19.5 mm, vias 0 -> 1
- net (no net): track 0.00 -> 7.65 mm
- net /Bemf_C: track 53.1 -> 45.5 mm
- net GNDREF: track 6.92 -> 10.0 mm
- net +3V3: track 25.9 -> 28.1 mm
- net /BW_SEL: track 37.5 -> 36.3 mm
- added copper zone on Power, net +3V3
- added copper zone on Power, net /VCC
- added copper zone on GND, net GNDREF
Other:
- board outline added: 92.5 x 62 mm
- board text added: "3,3V"
- board text added: "GND"
- board text added: "ZK-Spannung"

Commit message: _____________________ < Layout Groundplanes >  ---------------------       \                    / \  //\        \    |\___/|      /   \//  \\             /0  0  \__  /    //  | \ \            /     /  \/_/    //   |  \  \            @_^_@'/   \/_   //    |   \   \            //_^_/     \/_ //     |    \    \         ( //) |        \///      |     \     \       ( / /) _|_ /   )  //       |      \     _\     ( // /) '/,_ _ _/  ( ; -.    |    _ _\.-~        .-~~~^-.   (( / / )) ,-{        _      `-.|.-~-.           .~         `.  (( // / ))  '/\      /                 ~-. _ .-~      .-~^-.  \  (( /// ))      `.   {            }                   /      \  \   (( / ))     .----~-.\        \-'                 .~         \  `. \^-.              ///.----..>        \             _ -~             `.  ^-`  ^-_                ///-._ _ _ _ _ _ _}^ - - - - ~                     ~-- ,.-~                                                                   /.-~
Parts:
- removed C9: C, Capacitors_THT:CP_Radial_D10.0mm_P5.00mm
- moved C6 3.05 mm to (198.8, 62.5), turned to 270 degrees
- moved TP1 2.63 mm to (204.0, 49.5)
Connections:
- C1 pad 1: /Vin -> /VCC
- J6 pad 1: /Vin -> /VCC
Routing:
- net GNDREF: track 10.0 -> 103.8 mm, vias 5 -> 42
- net +3V3: track 28.1 -> 68.6 mm, vias 0 -> 20
- net /VCC: track 9.63 -> 28.2 mm, vias 0 -> 9
- net Net-(J5-Pad6): track 2.34 -> 16.9 mm
- net /Bemf_C: track 45.5 -> 53.1 mm
- net (no net): track 7.65 -> 0.00 mm
- added copper zone on F.Cu, net /VCC

Commit message: ___________ < remodeled >  -----------       \                    / \  //\        \    |\___/|      /   \//  \\             /0  0  \__  /    //  | \ \            /     /  \/_/    //   |  \  \            @_^_@'/   \/_   //    |   \   \            //_^_/     \/_ //     |    \    \         ( //) |        \///      |     \     \       ( / /) _|_ /   )  //       |      \     _\     ( // /) '/,_ _ _/  ( ; -.    |    _ _\.-~        .-~~~^-.   (( / / )) ,-{        _      `-.|.-~-.           .~         `.  (( // / ))  '/\      /                 ~-. _ .-~      .-~^-.  \  (( /// ))      `.   {            }                   /      \  \   (( / ))     .----~-.\        \-'                 .~         \  `. \^-.              ///.----..>        \             _ -~             `.  ^-`  ^-_                ///-._ _ _ _ _ _ _}^ - - - - ~                     ~-- ,.-~                                                                   /.-~
Parts:
- added C14: C, Capacitors_SMD:C_1812, F.Cu at (234.0, 58.0)
- added C15: C, Capacitors_SMD:C_1812, F.Cu at (252.5, 58.0)
- added C27: C, Capacitors_THT:CP_Radial_D10.0mm_P5.00mm, F.Cu at (209.5, 62.5)
- added C9: C, Capacitors_SMD:C_1812, F.Cu at (215.5, 58.0)
- added R11, R12, R14, R15, R8: R, Resistors_SMD:R_0603, F.Cu at (223.8, 90.1)
- R16: moved to B.Cu
- U7: value NC7WZ32 -> 74HC32D; footprint Housings_SSOP:VSSOP-8_2.3x2mm_Pitch0.5mm -> Housings_SSOP:TSSOP-14_4.4x5mm_Pitch0.65mm
- moved TP21 24.0 mm to (232.0, 75.0)
- moved U1 13.3 mm to (242.0, 74.7)
- moved TP11 11.6 mm to (257.0, 65.0)
- moved TP9 11.3 mm to (237.5, 65.0)
- moved TP7 10.3 mm to (219.0, 65.0)
- moved R42 10.1 mm to (204.0, 26.9), turned to 90 degrees
- moved R7 9.89 mm to (256.6, 77.5)
- moved J1 9.57 mm to (228.5, 58.0)
- moved Q6 9.39 mm to (259.0, 61.5), turned to 180 degrees
- moved Q4 9.23 mm to (222.0, 61.5), turned to 180 degrees
- moved Q5 9.19 mm to (240.5, 61.5), turned to 180 degrees
- moved J2 8.41 mm to (247.0, 58.0)
- moved R2 7.48 mm to (253.7, 76.4)
- moved J3 7.42 mm to (265.5, 58.0)
- moved C11 6.92 mm to (205.7, 26.9), turned to 90 degrees
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Connections:
- R22 pad 2: /Stop_Hardware -> Net-(R22-Pad2)
- U1 pad 10: (no net) -> Net-(R11-Pad2)
- U1 pad 11: (no net) -> Net-(R12-Pad2)
- U1 pad 13: (no net) -> /OVoltage
- U5 pad 1: /Stop_Hardware -> Net-(R22-Pad2)
- U7 pad 1: /Stop_Hardware -> /OR1
- U7 pad 3: Net-(R27-Pad2) -> /Stop
- U7 pad 4: GNDREF -> Net-(R22-Pad2)
- U7 pad 5: /Freigabe_button -> /OVoltage
- U7 pad 6: /Freigabe_MCU -> /OR1
- U7 pad 7: /Stop -> GNDREF
- U7 pad 8: +3V3 -> Net-(R27-Pad2)
Routing:
- net /Sternpunkt_virtuell: track 70.4 -> 0.00 mm, vias 2 -> 0
- net /Bemf_C: track 53.1 -> 6.74 mm, vias 3 -> 0
- net /Bemf_A: track 71.1 -> 29.4 mm
- net /A: track 54.0 -> 16.6 mm
- net /Bemf_B: track 55.3 -> 24.6 mm
- net /LO_A: track 21.3 -> 0.00 mm, vias 2 -> 0
- net /LO_C: track 20.7 -> 0.00 mm, vias 1 -> 0
- net /LO_B: track 19.5 -> 0.00 mm, vias 1 -> 0
- net /B: track 30.0 -> 17.1 mm
- net /C: track 35.2 -> 46.8 mm, vias 0 -> 1
- net /Stop_Hardware: track 11.4 -> 0.00 mm
- net Net-(R22-Pad2): track 0.00 -> 11.3 mm
- net (no net): track 0.00 -> 10.4 mm, vias 0 -> 3
- net Net-(R27-Pad2): track 11.5 -> 2.26 mm
- net /OR1: track 0.00 -> 8.75 mm, vias 0 -> 2
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- removed copper zone on F.Cu, net /A
- removed copper zone on F.Cu, net /B
- removed copper zone on F.Cu, net /C
- removed copper zone on F.Cu, net /Meas_out
- removed copper zone on B.Cu, net /Sternpunkt_virtuell

Commit message: ______________________ < Layout überarbeitet >  ----------------------       \                    / \  //\        \    |\___/|      /   \//  \\             /0  0  \__  /    //  | \ \            /     /  \/_/    //   |  \  \            @_^_@'/   \/_   //    |   \   \            //_^_/     \/_ //     |    \    \         ( //) |        \///      |     \     \       ( / /) _|_ /   )  //       |      \     _\     ( // /) '/,_ _ _/  ( ; -.    |    _ _\.-~        .-~~~^-.   (( / / )) ,-{        _      `-.|.-~-.           .~         `.  (( // / ))  '/\      /                 ~-. _ .-~      .-~^-.  \  (( /// ))      `.   {            }                   /      \  \   (( / ))     .----~-.\        \-'                 .~         \  `. \^-.              ///.----..>        \             _ -~             `.  ^-`  ^-_                ///-._ _ _ _ _ _ _}^ - - - - ~                     ~-- ,.-~                                                                   /.-~
Parts:
- R11, R12, R14, R15: moved to B.Cu
- moved R8 56.1 mm to (210.8, 35.5), turned to 270 degrees
- moved R11 43.6 mm to (261.6, 68.4), turned to 270 degrees
- moved R14 42.4 mm to (261.6, 71.1), turned to 270 degrees
- moved R2 39.8 mm to (262.2, 37.6), turned to 90 degrees
- moved R12 36.4 mm to (253.0, 68.4), turned to 270 degrees
- moved R15 34.9 mm to (253.0, 71.1), turned to 270 degrees
- moved R7 33.8 mm to (261.6, 44.0), turned to 180 degrees
- moved TP21 22.2 mm to (250.5, 62.8)
- moved R10 19.8 mm to (258.6, 42.7), turned to 180 degrees
- moved R4 12.2 mm to (265.5, 61.7), turned to 90 degrees
- moved C1 11.2 mm to (240.8, 70.3), turned to 180 degrees
- moved TP17 8.61 mm to (204.2, 71.9)
- moved U1 7.39 mm to (246.7, 69.0), turned to 0 degrees
- moved R3 3.91 mm to (247.0, 61.7)
- moved TP8 3.86 mm to (247.5, 52.6)
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Connections:
- C6 pad 1: (no net) -> /VCC
Routing:
- net /OVoltage: track 0.00 -> 109.8 mm, vias 0 -> 3
- net /Bemf_C: track 6.74 -> 72.3 mm, vias 0 -> 1
- net /Bemf_A: track 29.4 -> 92.0 mm
- net /Sternpunkt_virtuell: track 0.00 -> 59.9 mm
- net /Bemf_B: track 24.6 -> 78.3 mm
- net /A: track 16.6 -> 48.1 mm
- net /VCC: track 22.4 -> 47.4 mm, vias 8 -> 10
- net GNDREF: track 97.1 -> 117.4 mm, vias 36 -> 40
- net /B: track 17.1 -> 32.5 mm
- net /LO_B: track 0.00 -> 14.2 mm
- net Net-(R11-Pad2): track 0.00 -> 14.0 mm
- net /LO_C: track 0.00 -> 13.5 mm
- net /LO_A: track 0.00 -> 13.1 mm
- net /C: track 46.8 -> 38.1 mm, vias 1 -> 0
- net /Meas_out: track 4.14 -> 12.7 mm, vias 0 -> 3
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- added copper zone on F.Cu, net /A
- added copper zone on F.Cu, net /B
- added copper zone on F.Cu, net /C
- added copper zone on F.Cu, net /Meas_out

Commit message: ________________ < Mounting Holes >  ----------------       \                    / \  //\        \    |\___/|      /   \//  \\             /0  0  \__  /    //  | \ \            /     /  \/_/    //   |  \  \            @_^_@'/   \/_   //    |   \   \            //_^_/     \/_ //     |    \    \         ( //) |        \///      |     \     \       ( / /) _|_ /   )  //       |      \     _\     ( // /) '/,_ _ _/  ( ; -.    |    _ _\.-~        .-~~~^-.   (( / / )) ,-{        _      `-.|.-~-.           .~         `.  (( // / ))  '/\      /                 ~-. _ .-~      .-~^-.  \  (( /// ))      `.   {            }                   /      \  \   (( / ))     .----~-.\        \-'                 .~         \  `. \^-.              ///.----..>        \             _ -~             `.  ^-`  ^-_                ///-._ _ _ _ _ _ _}^ - - - - ~                     ~-- ,.-~                                                                   /.-~
Parts:
- added J10: Screw_Terminal_01x01, Mounting_Holes:MountingHole_3.2mm_M3_DIN965, F.Cu at (199.5, 77.0)
- added J11: Screw_Terminal_01x01, Mounting_Holes:MountingHole_3.2mm_M3_DIN965, F.Cu at (263.2, 77.0)
- added J8: Screw_Terminal_01x01, Mounting_Holes:MountingHole_3.2mm_M3_DIN965, F.Cu at (266.0, 21.2)
- added J9: Screw_Terminal_01x01, Mounting_Holes:MountingHole_3.2mm_M3_DIN965, F.Cu at (197.8, 37.0)
Routing:
- net /VCC: track 47.4 -> 56.1 mm, vias 10 -> 16
- net +3V3: track 69.0 -> 73.3 mm, vias 19 -> 21
- net (no net): track 6.22 -> 3.54 mm, vias 3 -> 1
- net GNDREF: track 117.4 -> 119.8 mm, vias 40 -> 41
- added copper zone on B.Cu, net /VCC
Other:
- board text added: "Freigabe"
- board text added: "Hochlauf"
- board text added: "PWR"
- board text added: "Stop"
- board text added: "el. Komm"

Commit message: Board fertig
Parts:
- removed J11: Screw_Terminal_01x01, Mounting_Holes:MountingHole_3.2mm_M3_DIN965
- added J12: Conn_01x01, kicadBibs:Führungsloch, F.Cu at (260.7, 78.7)
- added J13: Conn_01x01, kicadBibs:Führungsloch, F.Cu at (250.7, 78.6)
- added J14: Conn_01x01, kicadBibs:Führungsloch, F.Cu at (255.7, 78.6)
- R8: value R -> 10k
- moved C3 16.2 mm to (210.3, 47.4), turned to 180 degrees
- moved R6 14.5 mm to (210.3, 49.1), turned to 0 degrees
- moved R5 13.4 mm to (205.7, 53.1), turned to 270 degrees
- moved R13 7.70 mm to (238.5, 49.4), turned to 90 degrees
- moved D1 7.46 mm to (208.8, 53.1), turned to 90 degrees
- moved C7 7.26 mm to (240.2, 49.5)
- moved C10 6.59 mm to (262.5, 48.2), turned to 90 degrees
- moved Q10 6.10 mm to (253.6, 46.1)
- moved C2 5.97 mm to (211.2, 54.5)
- moved Q8 5.97 mm to (215.2, 47.1)
- moved U2 5.97 mm to (214.6, 53.2)
- moved U6 5.27 mm to (259.0, 48.5)
- moved D3 4.90 mm to (239.4, 58.2)
- moved C5 4.88 mm to (243.3, 56.9), turned to 0 degrees
- moved R9 3.05 mm to (235.4, 54.6)
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Routing:
- net /B: track 32.5 -> 22.3 mm
- net /HO_A: track 13.9 -> 20.5 mm, vias 1 -> 2
- net /A: track 48.1 -> 54.7 mm
- net /HI_A_F: track 25.7 -> 31.7 mm
- net /LI_A: track 27.5 -> 33.4 mm
- net /LO_C: track 13.5 -> 19.3 mm, vias 0 -> 1
- net /HO_B: track 16.0 -> 10.4 mm, vias 1 -> 0
- net Net-(C7-Pad1): track 8.64 -> 3.31 mm
- net Net-(C3-Pad1): track 10.8 -> 15.3 mm
- net Net-(C8-Pad1): track 4.60 -> 8.80 mm
- net /C: track 38.1 -> 42.3 mm
- net /LO_B: track 14.2 -> 18.3 mm, vias 0 -> 2
- net Net-(C5-Pad1): track 4.07 -> 0.00 mm
- net Net-(D3-Pad2): track 3.31 -> 0.00 mm
- net (no net): track 3.54 -> 0.76 mm
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- added copper zone on B.Cu, net /C
