File: Hardware/Elektrische_Komm.kicad_pcb (KiCad board)
At the start: 4 copper layers, 92.5 x 62 mm, 138 parts, among them J1 Conn_01x01, J10 Screw_Terminal_01x01, J12 Conn_01x01, J13 Conn_01x01, J14 Conn_01x01, J2 Conn_01x01, J3 Conn_01x01, J4 Conn_01x04, J5 USB_OTG, J6 Conn_01x01, J7 Conn_01x01, J8 Screw_Terminal_01x01, J9 Screw_Terminal_01x01, Q1 CSD16556Q5B, Q10 BSR202NL6327HTSA1, Q11 BSR202NL6327HTSA1, Q12 BSR202NL6327HTSA1, Q13 BSR202NL6327HTSA1, Q14 BSR202NL6327HTSA1, Q2 CSD16556Q5B, Q3 CSD16556Q5B, Q4 CSD16556Q5B, Q5 CSD16556Q5B, Q6 CSD16556Q5B, Q7 BSR202NL6327HTSA1, Q8 BSR202NL6327HTSA1, Q9 BSR202NL6327HTSA1, SW1 SW_Push, SW2 SW_Push, U1 TS374IDT, U10 TPS561201, U12 STM32F413R(G-H)Tx_u, U2 UCC27710, U3 ACS723LLCTR, U4 UCC27710, U5 MCP6546, U6 UCC27710, U7 74HC32D, U8 74LVC2G02, Y1 24MHz

Commit message: _________________________ < Zener-Spannungsreferenz >  -------------------------       \                    / \  //\        \    |\___/|      /   \//  \\             /0  0  \__  /    //  | \ \            /     /  \/_/    //   |  \  \            @_^_@'/   \/_   //    |   \   \            //_^_/     \/_ //     |    \    \         ( //) |        \///      |     \     \       ( / /) _|_ /   )  //       |      \     _\     ( // /) '/,_ _ _/  ( ; -.    |    _ _\.-~        .-~~~^-.   (( / / )) ,-{        _      `-.|.-~-.           .~         `.  (( // / ))  '/\      /                 ~-. _ .-~      .-~^-.  \  (( /// ))      `.   {            }                   /      \  \   (( / ))     .----~-.\        \-'                 .~         \  `. \^-.              ///.----..>        \             _ -~             `.  ^-`  ^-_                ///-._ _ _ _ _ _ _}^ - - - - ~                     ~-- ,.-~                                                                   /.-~
Parts:
- removed R14: R, Resistors_SMD:R_0603
- added D2: D_Zener, Diodes_SMD:D_SOD-323, B.Cu at (260.6, 71.9)
- C10, C3, C7: footprint Capacitors_SMD:C_0603 -> Capacitors_SMD:C_0805
- C13: footprint Capacitors_SMD:C_1206 -> Capacitors_SMD:C_0805
- R11: value R -> 200k
- R12: value R -> 612k
- R15: value R -> 100k
- R35, R36, R37, R38, R39: value R -> 100
- moved C7 3.84 mm to (236.3, 49.4)
- moved C3 0.79 mm to (209.6, 47.1)
- moved TP5 0.28 mm to (264.4, 47.8)
- moved C10 0.26 mm to (262.6, 48.0)
Routing:
- net Net-(C3-Pad1): track 15.3 -> 4.95 mm
- net Net-(C7-Pad1): track 3.31 -> 5.77 mm
- net /LI_B: track 21.6 -> 20.1 mm, vias 3 -> 2
- net Net-(D2-Pad1): track 14.0 -> 15.5 mm
- net GNDREF: track 118.1 -> 116.7 mm
- net /VCC: track 54.4 -> 55.2 mm, vias 15 -> 16
- net (no net): track 0.76 -> 1.37 mm

Commit message: ________________________ < Gerber-Files geplottet >  ------------------------       \                    / \  //\        \    |\___/|      /   \//  \\             /0  0  \__  /    //  | \ \            /     /  \/_/    //   |  \  \            @_^_@'/   \/_   //    |   \   \            //_^_/     \/_ //     |    \    \         ( //) |        \///      |     \     \       ( / /) _|_ /   )  //       |      \     _\     ( // /) '/,_ _ _/  ( ; -.    |    _ _\.-~        .-~~~^-.   (( / / )) ,-{        _      `-.|.-~-.           .~         `.  (( // / ))  '/\      /                 ~-. _ .-~      .-~^-.  \  (( /// ))      `.   {            }                   /      \  \   (( / ))     .----~-.\        \-'                 .~         \  `. \^-.              ///.----..>        \             _ -~             `.  ^-`  ^-_                ///-._ _ _ _ _ _ _}^ - - - - ~                     ~-- ,.-~                                                                   /.-~
Parts:
- added R14: 1k, Resistors_SMD:R_0603, F.Cu at (201.9, 37.5)
- added SW3: SW_Push, kicadBibs:Switch, F.Cu at (198.0, 43.7)
- added TP26: TEST, Pin_Headers:Pin_Header_Straight_1x01_Pitch1.00mm, F.Cu at (224.6, 50.0)
- D2: value D_Zener -> MM3Z5V6T1G
- R11: value 200k -> 9,4k
- R12: value 612k -> 523k
- R16: value R -> 100k
Connections:
- U12 pad 52: (no net) -> /StopButton
Routing:
- net /StopButton: track 0.00 -> 77.7 mm
- net GNDREF: track 116.7 -> 125.6 mm, vias 41 -> 42
- net +3V3: track 73.1 -> 74.3 mm, vias 21 -> 22
- added copper zone on F.Cu, net Net-(C12-Pad2)
Other:
- board text added: "VCC"

Commit message: __________________________ < Messstation hinzugefügt >  --------------------------       \                    / \  //\        \    |\___/|      /   \//  \\             /0  0  \__  /    //  | \ \            /     /  \/_/    //   |  \  \            @_^_@'/   \/_   //    |   \   \            //_^_/     \/_ //     |    \    \         ( //) |        \///      |     \     \       ( / /) _|_ /   )  //       |      \     _\     ( // /) '/,_ _ _/  ( ; -.    |    _ _\.-~        .-~~~^-.   (( / / )) ,-{        _      `-.|.-~-.           .~         `.  (( // / ))  '/\      /                 ~-. _ .-~      .-~^-.  \  (( /// ))      `.   {            }                   /      \  \   (( / ))     .----~-.\        \-'                 .~         \  `. \^-.              ///.----..>        \             _ -~             `.  ^-`  ^-_                ///-._ _ _ _ _ _ _}^ - - - - ~                     ~-- ,.-~                                                                   /.-~
Parts:
- added D11: BZT52-C3V0X, Diodes_SMD:D_SOD-123, B.Cu at (266.4, 53.5)
- added D12: BZT52-C3V0X, Diodes_SMD:D_SOD-123, B.Cu at (252.8, 61.3)
- added D13: BZT52-C3V0X, Diodes_SMD:D_SOD-123, B.Cu at (234.4, 62.7)
- added D14: BZT52-C3V0X, Diodes_SMD:D_SOD-123, B.Cu at (230.4, 53.0)
- added R20: 4M, Resistors_SMD:R_0603, B.Cu at (264.2, 54.9)
- added R21: 4M, Resistors_SMD:R_0603, B.Cu at (250.3, 58.0)
- added R28: 4M, Resistors_SMD:R_0603, B.Cu at (234.8, 65.5)
- added R32: 4M, Resistors_SMD:R_0603, B.Cu at (228.4, 54.7)
- added R33: 1M, Resistors_SMD:R_0603, B.Cu at (262.3, 54.9)
- added R34: 1M, Resistors_SMD:R_0603, B.Cu at (250.3, 59.8)
- added R40: 1M, Resistors_SMD:R_0603, B.Cu at (232.9, 65.5)
- added R43: 1M, Resistors_SMD:R_0603, B.Cu at (228.4, 51.7)
Connections:
- U12 pad 10: (no net) -> /Me_B
- U12 pad 11: (no net) -> /Me_C
- U12 pad 8: (no net) -> /Me_A
- U12 pad 9: (no net) -> /Me_VS
Routing:
- net /Me_C: track 0.00 -> 47.7 mm, vias 0 -> 4
- net /Me_B: track 0.00 -> 40.6 mm, vias 0 -> 5
- net /Me_VS: track 0.00 -> 40.2 mm, vias 0 -> 5
- net /Me_A: track 0.00 -> 33.4 mm, vias 0 -> 7
- net GNDREF: track 125.6 -> 136.1 mm, vias 42 -> 50
- net /C: track 42.3 -> 45.1 mm
- net /A: track 54.7 -> 57.3 mm
- net /B: track 22.3 -> 24.9 mm
- net /Meas_out: track 12.7 -> 14.7 mm
- net /Sternpunkt_virtuell: track 59.8 -> 61.5 mm
Other:
- board text added: "Brückenspannung"
- board text added: "Sensorlose Elektrische Kommutierung SoSe 2018 Stefan Waldmann"
- board text removed: "ZK-Spannung"

Commit message: _______ < jetzt >  -------       \                    / \  //\        \    |\___/|      /   \//  \\             /0  0  \__  /    //  | \ \            /     /  \/_/    //   |  \  \            @_^_@'/   \/_   //    |   \   \            //_^_/     \/_ //     |    \    \         ( //) |        \///      |     \     \       ( / /) _|_ /   )  //       |      \     _\     ( // /) '/,_ _ _/  ( ; -.    |    _ _\.-~        .-~~~^-.   (( / / )) ,-{        _      `-.|.-~-.           .~         `.  (( // / ))  '/\      /                 ~-. _ .-~      .-~^-.  \  (( /// ))      `.   {            }                   /      \  \   (( / ))     .----~-.\        \-'                 .~         \  `. \^-.              ///.----..>        \             _ -~             `.  ^-`  ^-_                ///-._ _ _ _ _ _ _}^ - - - - ~                     ~-- ,.-~                                                                   /.-~
Other:
- board text added: "Sensorlose Elektrische Kommutierung SoSe 2018 -Abschluss Stefan Waldmann"
- board text removed: "Sensorlose Elektrische Kommutierung SoSe 2018 Stefan Waldmann"
Changed lines of the file:
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@@
     (links 428)
     (no_connects 0)
-    (area 177.449999 17.949999 270.050001 80.050001)
+    (area 173.262999 12.97569 274.628573 81.875)
     (thickness 1.6)
     (drawings 53)
@@
     )
   )
-  (gr_text "Sensorlose Elektrische Kommutierung\nSoSe 2018\nStefan Waldmann" (at 210.6168 73.4314) (layer F.SilkS)
+  (gr_text "Sensorlose Elektrische Kommutierung\nSoSe 2018 -Abschluss\nStefan Waldmann\n\n" (at 210.6168 73.4314) (layer F.SilkS)
     (effects (font (size 1.5 1.5) (thickness 0.3)) (justify left))
   )
